File: OudOntwerp/Load.sch (KiCad schematic (older format))
At the start: 12 parts, among them Q1 BC547, Q2 BC547, Q3 BC547, Q4 2N3773

Commit message: Sync_21-04-27
Parts:
- R2: value 33R -> 120R
- R5: value 0,5R -> 0R33
- RV1: symbol Device:R_POT -> Device:R_Potentiometer
Changed lines of the file:
@@
 P 6250 4150
 F 0 "R5" H 6320 4196 50  0000 L CNN
-F 1 "0,5R" H 6320 4105 50  0000 L CNN
+F 1 "0R33" H 6320 4105 50  0000 L CNN
 F 2 "" V 6180 4150 50  0001 C CNN
 F 3 "~" H 6250 4150 50  0001 C CNN
@@
 $EndComp
 $Comp
-L Device:R_POT RV1
+L Device:R_Potentiometer RV1
 U 1 1 5F9EFD91
 P 5500 3600
@@
 P 4850 4150
 F 0 "R2" H 4920 4196 50  0000 L CNN
-F 1 "33R" H 4920 4105 50  0000 L CNN
+F 1 "120R" H 4920 4105 50  0000 L CNN
 F 2 "" V 4780 4150 50  0001 C CNN
 F 3 "~" H 4850 4150 50  0001 C CNN
