File: NieuwOntwerp/Load.sch (KiCad schematic (older format))
At the start: 74 parts, among them J1 Conn_01x02, J2 Conn_01x02, J3 Conn_01x05, J4 Conn_01x03, J5 Conn_01x02, Q1 IRF840, Q2 IRF840, T1 EE13, U1 ESP12E, U10 MCP4725A0, U2 LNK364D, U3 LM358, U4 PC817, U5 TL431, U6 LM1117-3.3, U7 LM358

Commit message: --
Parts:
- Q1, Q2: Spice_Lib_File (none) -> C:\\Users\\Erik\\Documents\\Elektronika\\2021\\AdjustableCu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; Spice_Model (none) -> irf840; Spice_Netlist_Enabled (none) -> Y; Spice_Primitive (none) -> Q
Changed lines of the file:
@@
 $Descr A4 11693 8268
 encoding utf-8
-Sheet 1 2
+Sheet 1 3
 Title "Adjustable Current"
 Date "2021-01-28"
@@
 F 2 "Package_TO_SOT_THT:TO-220-3_Vertical" H 9250 4100 50  0001 C CNN
 F 3 "https://www.vishay.com/docs/91071/sihf840s.pdf" H 9050 4000 50  0001 C CNN
+F 4 "Q" H 9050 4000 50  0001 C CNN "Spice_Primitive"
+F 5 "irf840" H 9050 4000 50  0001 C CNN "Spice_Model"
+F 6 "Y" H 9050 4000 50  0001 C CNN "Spice_Netlist_Enabled"
+F 7 "C:\\Users\\Erik\\Documents\\Elektronika\\2021\\AdjustableCurrentLoad\\Spice\\Lib\\IRF840.lib" H 9050 4000 50  0001 C CNN "Spice_Lib_File"
 	1    9050 4000
 	1    0    0    -1
@@
 F 2 "Package_TO_SOT_THT:TO-220-3_Vertical" H 10500 4100 50  0001 C CNN
 F 3 "https://www.vishay.com/docs/91071/sihf840s.pdf" H 10300 4000 50  0001 C CNN
+F 4 "Q" H 10300 4000 50  0001 C CNN "Spice_Primitive"
+F 5 "irf840" H 10300 4000 50  0001 C CNN "Spice_Model"
+F 6 "Y" H 10300 4000 50  0001 C CNN "Spice_Netlist_Enabled"
+F 7 "C:\\Users\\Erik\\Documents\\Elektronika\\2021\\AdjustableCurrentLoad\\Spice\\Lib\\IRF840.lib" H 10300 4000 50  0001 C CNN "Spice_Lib_File"
 	1    10300 4000
 	1    0    0    -1
@@
 Wire Wire Line
 	5750 1550 6150 1550
+$Sheet
+S 6150 7150 750  550
+U 601C1496
+F0 "SPICE" 50
+F1 "SPICE.sch" 50
+$EndSheet
 $EndSCHEMATC

Commit message: Sync_21-04-27
Parts:
- removed C10, C11, C14, C16: 100n, Capacitor_SMD:C_0603_1608Metric, symbol Device:C
- removed C12: 100nF, Capacitor_SMD:C_0603_1608Metric, symbol Device:C
- removed C13: 100uF/25V, Capacitor_THT:CP_Radial_D5.0mm_P2.00mm, symbol Device:C_Polarized
- removed C15: 10nF, Capacitor_SMD:C_0603_1608Metric, symbol Device:C
- removed C17: X type 470pF, Capacitor_SMD:C_0603_1608Metric, symbol Device:C
- removed C2: 4,7uF/400V, Capacitor_THT:CP_Radial_D8.0mm_P3.50mm, symbol Device:C_Polarized
- removed C3: 6,8uF/400V, Capacitor_THT:CP_Radial_D8.0mm_P3.50mm, symbol Device:C_Polarized
- removed C4: 1nF/300V, Condensator:JN_102M, symbol Device:C
- removed C8: 1000uF/25V, Capacitor_THT:CP_Radial_D10.0mm_P5.00mm, symbol Device:C_Polarized
- removed C9: 470pF/50V, Capacitor_SMD:C_0603_1608Metric, symbol Device:C
- removed D2: DB207S, Diode2:SOT4_Rectifier_Bridge, symbol Device:D_Bridge_+-AA
- removed D4: SS34, Diode_SMD:D_SMA, symbol Device:D
- removed F1: 0,3Amp, Fuse:Fuse_1206_3216Metric, symbol Device:Fuse
- removed J1: Conn_01x02, Connector2:JST_XH_B3B-XH-AM_1x03_P2.50mm_Vertical, symbol Connector_Generic:Conn_01x03
- removed J2, J5: Conn_01x02, Connector2:JST_XH_B2B-XH-AM_1x02_P2.50mm_Vertical, symbol Connector_Generic:Conn_01x02
- removed J3: Conn_01x05, Connector2:Molex_PicoBlade_53047-0510_1x05_P1.25mm_Vertical, symbol Connector_Generic:Conn_01x05
- removed J4: Conn_01x03, Connector2:JST_XH_B3B-XH-AM_1x03_P2.50mm_Vertical, symbol Connector_Generic:Conn_01x03
- removed L1: 6mH, Transformers:UU98_Common_Mode_Choke, symbol Device:L_Iron_Coupled_1423
- removed L2: 3,3uH, Inductor_SMD:L_1206_3216Metric, symbol Device:L
- removed R14: 22k, Resistor_SMD:R_0402_1005Metric, symbol Device:R
- removed RV1: 10D431K, Varistor2:RV_Disc_D10mm_W2mm_P8mm, symbol Device:Varistor
- removed RV2: 10K, Potentiometer_THT:Potentiometer_Bourns_3296W_Vertical, symbol Device:R_Potentiometer_Trim
- removed T1: EE13, Transformers:EE13Horizontal, symbol Device:Transformer_1P_1S
- removed U2: LNK364D, Package_SO:PowerIntegrations_SO-8C, symbol Regulator_Switching:LNK364D
- removed unit 3 of U3
- removed U4: PC817, Package_SO:SSO-4_6.7x5.1mm_P2.54mm_Clearance8mm, symbol Isolator:PC817
- removed U5: TL431, Package_TO_SOT_SMD:SOT-23, symbol Reference_Voltage:TL431DBZ
- removed U6: LM1117-3.3, Package_TO_SOT_SMD:SOT-223-3_TabPin2, symbol Regulator_Linear:LM1117-3.3
- added C2: 47pF, Capacitor_SMD:C_0603_1608Metric, symbol Device:C
- added C3: 10nF, Capacitor_SMD:C_0402_1005Metric, symbol Device:C
- added C?: C_Polarized, symbol Device:C_Polarized
- added D11, D2: LED, LED_SMD:LED_0603_1608Metric, symbol Device:LED
- added D?: 3V, symbol Device:D_Zener
- added FB1: 1K, Resistor_SMD:R_0603_1608Metric, symbol Device:FerriteBead
- added HS3: Heatsink, Mechanisch:Heatsink_TO220, symbol Mechanical:Heatsink
- added J1: USB_C_Receptacle_USB2.0, Connector2:USB-C_Receptable_SMD_16pin, symbol Connector:USB_C_Receptacle_USB2.0
- added J2: Conn_01x02, Connector2:JST_XH_B2B-XH-AM_1x02_P2.50mm_Vertical, symbol Connector_Generic:Conn_01x04
- added Q3: 4809NG, Package-SOT:369AA, symbol Device:Q_NMOS_GDS
- added Q4: IRF840, Package_TO_SOT_THT:TO-220-3_Vertical, symbol Device:Q_NMOS_GDS
- added R17, R37, R42: 100K, Resistor_SMD:R_0603_1608Metric, symbol Device:R
- added R33: 33K, Resistor_SMD:R_0603_1608Metric, symbol Device:R
- added R35: 10K, Resistor_SMD:R_0603_1608Metric, symbol Device:R
- added R36: 0R, Resistor_SMD:R_0603_1608Metric, symbol Device:R
- added R38, R39: 27R, Resistor_SMD:R_0603_1608Metric, symbol Device:R
- added R40, R41: 1K6, Resistor_SMD:R_0603_1608Metric, symbol Device:R
- added R43: 470R, Resistor_SMD:R_0603_1608Metric, symbol Device:R
- added R44: 100k, Resistor_SMD:R_0603_1608Metric, symbol Device:R
- added R45, R6: 0R002, Resistor_SMD:R_1206_3216Metric, symbol Device:R
- added R?: ??, Resistor_SMD:R_0603_1608Metric, symbol Device:R
- added TH3: 10k_NTC, Capacitor_THT:C_Disc_D3.8mm_W2.6mm_P2.50mm, symbol Device:Thermistor_NTC
- added U13: FT231XQ, Package_DFN_QFN:QFN-20-1EP_4x4mm_P0.5mm_EP2.5x2.5mm, symbol Interface_USB:FT231XQ
- added unit 1 of U2
- added U3: LM358, Package_SO:SOIC-8_3.9x4.9mm_P1.27mm, symbol Amplifier_Operational:LM358
- C1: value X2 100nF/275V -> 470pF; footprint Condensator:CBB22104J400V -> Capacitor_SMD:C_0402_1005Metric
- C5: value Y type 2N2/250VAC -> 47pF; footprint Condensator:JN_102M -> Capacitor_SMD:C_0603_1608Metric
- C6: value 100nF/50V -> 100nF
- C7: value Y type 2N2/250VAC -> 100n; footprint Condensator:JN_102M -> Capacitor_SMD:C_0603_1608Metric
- D3: value FR107 -> SMA12JA
- R1: value 5k6 -> 100K; footprint Resistor_SMD:R_0603_1608Metric_Pad1.05x0.95mm_HandSolder -> Resistor_SMD:R_0603_1608Metric
- R11: value 18R -> 1K8; footprint Resistor_SMD:R_1206_3216Metric -> Resistor_SMD:R_0603_1608Metric
- R12: value 150 -> ??
- R13: value 1K -> 100K
- R15: value 6K8 -> 56K
- R16, R19, R2, R22, R23, R3: footprint Resistor_SMD:R_0603_1608Metric_Pad1.05x0.95mm_HandSolder -> Resistor_SMD:R_0603_1608Metric
- R4: value 2K2 -> 100K
- R5: value 10R -> 0R002; footprint Resistor_SMD:R_2512_6332Metric -> Resistor_SMD:R_1206_3216Metric
- R7: value 300R -> 100K; footprint Resistor_SMD:R_1210_3225Metric -> Resistor_SMD:R_0603_1608Metric
- R8: value 100k -> 10K; footprint Resistor_SMD:R_1210_3225Metric -> Resistor_SMD:R_0603_1608Metric
- U7: value LM358 -> (none)
- renumbered U3 to U2
Connections:
- net +3V3: now also R1.2, C?.1, TH3.1
- net DTR: now also U13.18 (~DTR)
- net GND: now also C5.2, C6.2, C7.1, R13.1, C2.2, C3.2, J1.A1 (GND), J1.A12 (GND), J1.B1 (GND), J1.B12 (GND), J1.S1 (SHIELD), R33.1, R37.1, U13.13 (GND), U13.21 (GND), U13.3 (GND); no longer R1.2, R15.2, R4.2
- net LOAD: now also Q4.2 (D)
- net RTS: now also U13.19 (~RTS)
- net SHUNT: now also R5.1, R45.1, R6.1; no longer Q1.3 (S), Q2.3 (S), R19.2, R23.2
- net THERM: now also R12.2, C?.2, TH3.2, U3.6 (-); no longer R1.1, U1.2 (ADC)
- net GNDA: now reaches C1.1
- net GNDA: now also R12.1, R7.1; no longer R5.1
- net at R5.2: now also Q1.3 (S), R19.2; no longer C5.2
- net at R8.1: now also R1.1, R7.2, U3.3 (+)
- net at C6.1: now also U13.10 (3V3OUT), U13.11 (~RESET), U13.20 (VCCIO)
- net at D3.2 (A): now also J2.4 (Pin_4), Q3.2 (D), R?.1
- net at R13.2: now also R15.2, U2.2 (-)
- net at R11.2: now also R8.2, U3.1
- net at R15.1: now also R35.2, U2.1
- net +12V: now reaches D3.1 (K)
- net +12V: now also J2.2 (Pin_2), R17.2, R?.2; no longer R7.2
- net at R11.1: now also C1.2, U3.2 (-), U3.5 (+)
- net at R16.1, R22.1: now also R4.1, U2.7, R43.1; no longer U2.1
- net at U10.1 (VOUT): now also U2.3 (+); no longer U2.3 (+)
- net TX: now reaches U1.16 (TXD)
- net TX: now also U13.1 (RXD)
- net RX: now reaches U1.15 (RXD)
- net RX: now also U13.17 (TXD)
- net FAN_TACH: now reaches U1.5 (GPIO14)
- net FAN_TACH: now also D?.1 (K), J2.3 (Pin_3)
- net Earth: no longer names the net of C5.1
- net Earth: now also J1.A6 (D+), J1.B6 (D+), R39.2; no longer C7.2
- removed net NEUTRAL: C1.2, C7.1
- new net: R35.1, R36.2, U2.5 (+)
- new net: R37.2, R4.2, U2.6 (-)
- new net: Q2.3 (S), R23.2, R6.2
- new net: C3.1, FB1.2, J1.A4 (VBUS), J1.A9 (VBUS), J1.B4 (VBUS), J1.B9 (VBUS)
- new net: C2.1, J1.A7 (D-), J1.B7 (D-), R38.2
- new net: D11.1 (K), U13.14 (CBUS1)
- new net: D2.1 (K), U13.7 (CBUS2)
- new net: R39.1, U13.8 (USBDP)
- new net: R38.1, U13.9 (USBDM)
- new net: D11.2 (A), R40.1
- new net: D2.2 (A), R41.1
- new net: C7.2, Q4.1 (G), R43.2, R44.1
- new net: Q4.3 (S), R44.2, R45.2
- new net: R17.1, R33.2, R36.1
- new net: Q3.1 (G), R42.2, U3.7
- new net: D?.2 (A), J2.1 (Pin_1), Q3.3 (S), R42.1
- new net VCC: FB1.1, R40.2, R41.2, U13.12 (VCC)
- no-connect marks 10 -> 20
Other:
- note added: "+12V"
- note added: "FAN"
- note added: "GND"
- note added: "Green"
- note added: "MOSFET, max power, 1x 125W with Heatsink"
- note added: "PWM"
- note added: "PWM FAN Control"
- note added: "Programming Interface"
- note added: "TACH"
- note added: "VOLT Measure"
- note added: "Yellow"
- note removed: "12V"
- note removed: "230V AC"
- note removed: "Connections to case"
- note removed: "Connectors to Front Panel"
- note removed: "MOSFET, max power, 2x 125W with Heatsink"
- note removed: "Power Supply"
- note removed: "place as close as possible to the supply and ground pins."
- moved on the sheet: C18, C19, C20, D1, H1, H2, H3, H4, HS1, HS2, Q1, Q2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

Commit message: 2021-04-27_02
Parts:
- added D?: 3V, symbol Device:D_Zener
- added R?: 10k, Resistor_SMD:R_0603_1608Metric, symbol Device:R
- R2: value 10k -> 330K
Connections:
- net +3V3: no longer R2.1
- net GND: now also D?.2 (A), R?.2
- net LOAD: now also R2.1
- net RTS: no longer R2.2
- net ADC: now reaches U1.2 (ADC)
- net ADC: now also R2.2, D?.1 (K), R?.1
Other:
- moved on the sheet: R2
Changed lines of the file:
@@
 L Device:R R2
 U 1 1 6015AC04
-P 1200 1050
-F 0 "R2" H 1000 1100 50  0000 L CNN
-F 1 "10k" V 1200 1000 50  0000 L CNN
-F 2 "Resistor_SMD:R_0603_1608Metric" V 1130 1050 50  0001 C CNN
-F 3 "~" H 1200 1050 50  0001 C CNN
-	1    1200 1050
-	1    0    0    -1
-$EndComp
-Wire Wire Line
-	1200 1200 1200 1350
+P 900 3450
+F 0 "R2" H 700 3500 50  0000 L CNN
+F 1 "330K" V 900 3350 50  0000 L CNN
+F 2 "Resistor_SMD:R_0603_1608Metric" V 830 3450 50  0001 C CNN
+F 3 "~" H 900 3450 50  0001 C CNN
+	1    900  3450
+	1    0    0    -1
+$EndComp
 Wire Wire Line
 	1350 1150 1350 900
@@
 Wire Notes Line
 	4400 4700 11050 4700
-Wire Notes Line
-	600  3050 2900 3050
-Wire Notes Line
-	2900 3050 2900 4550
-Wire Notes Line
-	2900 4550 600  4550
-Wire Notes Line
-	600  4550 600  3050
-Text Notes 1550 3800 0    50   ~ 0
+Text Notes 650  3150 0    50   ~ 0
 VOLT Measure
 Wire Wire Line
@@
 Connection ~ 5450 1200
 Connection ~ 6300 1700
+$Comp
+L Device:R R?
+U 1 1 6088EF1E
+P 900 3750
+F 0 "R?" H 700 3800 50  0000 L CNN
+F 1 "10k" V 900 3650 50  0000 L CNN
+F 2 "Resistor_SMD:R_0603_1608Metric" V 830 3750 50  0001 C CNN
+F 3 "~" H 900 3750 50  0001 C CNN
+	1    900  3750
+	1    0    0    -1
+$EndComp
+Text GLabel 1200 3600 2    50   Input ~ 0
+ADC
+Text GLabel 1350 1250 0    50   Input ~ 0
+ADC
+$Comp
+L Device:D_Zener D?
+U 1 1 6088FDD6
+P 1100 3750
+F 0 "D?" V 1000 3750 50  0000 L CNN
+F 1 "3V" V 1200 3750 50  0000 L CNN
+F 2 "" H 1100 3750 50  0001 C CNN
+F 3 "~" H 1100 3750 50  0001 C CNN
+	1    1100 3750
+	0    1    1    0
+$EndComp
+$Comp
+L power:GND #PWR?
+U 1 1 60890C03
+P 900 3900
+F 0 "#PWR?" H 900 3650 50  0001 C CNN
+F 1 "GND" H 905 3727 50  0000 C CNN
+F 2 "" H 900 3900 50  0001 C CNN
+F 3 "" H 900 3900 50  0001 C CNN
+	1    900  3900
+	1    0    0    -1
+$EndComp
+Wire Wire Line
+	1200 3600 1100 3600
+Connection ~ 900  3600
+Connection ~ 1100 3600
+Wire Wire Line
+	1100 3600 900  3600
+Text GLabel 1200 3300 2    50   Input ~ 0
+LOAD
+Wire Wire Line
+	1200 3300 900  3300
+Wire Wire Line
+	1100 3900 900  3900
+Connection ~ 900  3900
+Wire Notes Line
+	600  3050 1500 3050
+Wire Notes Line
+	1500 3050 1500 4150
+Wire Notes Line
+	1500 4150 600  4150
+Wire Notes Line
+	600  3050 600  4150
 $EndSCHEMATC

Commit message: 2021-05-13_01
Parts:
- removed C?: C_Polarized, symbol Device:C_Polarized
- removed D?: 3V, symbol Device:D_Zener
- removed R12: ??, Resistor_SMD:R_0603_1608Metric, symbol Device:R
- added C5: 100uF, Capacitor_THT:CP_Radial_D6.3mm_P2.50mm, symbol Device:C_Polarized
- added D3: 1N4148, Diode2:DIO_LL4148, symbol Device:D
- added J?: Conn_01x02, Connector2:JST_XH_B2B-XH-AM_1x02_P2.50mm_Vertical, symbol Connector_Generic:Conn_01x02
- added Q1, Q?: Si2306, Package_TO_SOT_SMD:SOT-23, symbol Device:Q_NMOS_GSD
- added R6: 1K, Resistor_SMD:R_0603_1608Metric, symbol Device:R
- added R7: 56K, Resistor_SMD:R_0603_1608Metric, symbol Device:R
- added R?: 4K7, Resistor_SMD:R_0603_1608Metric, symbol Device:R
- added RV1: 10K, Potentiometer_THT:Potentiometer_Bourns_3266Y_Vertical, symbol Device:R_Potentiometer_Trim
- D1: renamed from D?; footprint (none) -> Diode_SMD:D_SMA
- R24: renamed from R?; value ?? -> 1K
- TH1, TH2, TH3: footprint Capacitor_THT:C_Disc_D3.8mm_W2.6mm_P2.50mm -> Thermistor:THERM_NXRT15XH103FA1B040
- gave numbers to parts that had none: 1
- renumbered C2 to C1, C7 to C10, C3 to C2, C5 to C3, C6 to C4, C1 to C6, C18 to C7, C20 to C8, C19 to C9, D1 to D2, D11 to D4, D2 to D5, D3 to D6, Q3 to Q2, Q1 to Q3, Q2 to Q4, Q4 to Q5, R2 to R1, R1 to R10, R7 to R11, R40 to R12, R41 to R13, R8 to R14, R11 to R15, R13 to R16, R15 to R17, R17 to R18, R33 to R19, R42 to R20, R35 to R21, R36 to R22, R37 to R23, R4 to R25, R16 to R26, R19 to R27, R5 to R28, R22 to R29, R23 to R30, R18 to R31, R6 to R32, R20 to R33, R21 to R34, R43 to R35, R44 to R36, R45 to R37, R38 to R4, R39 to R5, R9 to R8, R10 to R9, U13 to U2, U10 to U4, U2 to U5, U7 to U6
Connections:
- net +12V: now also J?.1 (Pin_1)
- net +3V3: now also C5.1, R?.2; no longer R10.2, TH1.1, TH2.1, TH3.1
- net FAN_TACH: now also R?.1
- net GND: now also TH1.2, TH2.2, TH3.2, D3.2 (A), Q1.2 (S), Q?.2 (S), R7.1
- net THERM: now also TH1.1, TH2.1, TH3.1, Q1.3 (D), Q?.3 (D), RV1.3; no longer TH1.2, TH2.2, TH3.2
- net FAN_OVERRIDE: now reaches U1.6 (GPIO12)
- net FAN_OVERRIDE: now also Q?.1 (G)
- net at D6.2 (A), J2.4 (Pin_4), Q2.2 (D)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: now also J?.2 (Pin_2)
- net GNDA: no longer names the net of C6.1, R11.1
- new net: C5.2, Q1.1 (G), R6.2, R7.2
- new net: D3.1 (K), R6.1
- new net +5V: R10.2, RV1.2
- no-connect marks 20 -> 18
Other:
- note added: "Fan start"

Commit message: 2021-05-14_01
Parts:
- added D?: D_Zener, symbol Device:D_Zener
- added R?: 4K7, Resistor_SMD:R_0603_1608Metric, symbol Device:R
- R?: value 4K7 -> 10K
Connections:
- net FAN_TACH: now also R?.2; no longer J2.3 (Pin_3), R?.1
- net GND: now also J2.1 (Pin_1), Q2.3 (S), R20.1, D?.2 (A)
- new net: D?.1 (K), J2.3 (Pin_3), R?.1, R?.1
Other:
- moved on the sheet: R?
Changed lines of the file:
@@
 	6600 1450 6800 1450
 Connection ~ 6600 1450
-Text GLabel 7350 2200 2    50   Input ~ 0
+Text GLabel 7950 1900 2    50   Input ~ 0
 FAN_TACH
 $Comp
@@
 	4400 2300 7800 2300
 Wire Notes Line
-	7800 2300 7800 650
+	8450 2300 8450 650
 Wire Notes Line
 	7800 650  4400 650
@@
 Connection ~ 6800 1450
 Wire Wire Line
-	7000 1750 7000 2100
-Wire Wire Line
 	4850 1600 5450 1600
 Connection ~ 5450 1600
@@
 	2400 3650 2400 3700
 Wire Wire Line
-	6600 2100 7000 2100
+	6600 2100 6700 2100
 $Comp
 L Device:Q_NMOS_GSD Q?
@@
 L Device:R R?
 U 1 1 60A70C52
-P 7300 2050
-F 0 "R?" H 7100 2100 50  0000 L CNN
-F 1 "4K7" V 7300 2000 50  0000 L CNN
-F 2 "Resistor_SMD:R_0603_1608Metric" V 7230 2050 50  0001 C CNN
-F 3 "~" H 7300 2050 50  0001 C CNN
-	1    7300 2050
-	-1   0    0    1
+P 7100 2000
+F 0 "R?" V 7200 2050 50  0000 L CNN
+F 1 "10K" V 7100 1950 50  0000 L CNN
+F 2 "Resistor_SMD:R_0603_1608Metric" V 7030 2000 50  0001 C CNN
+F 3 "~" H 7100 2000 50  0001 C CNN
+	1    7100 2000
+	0    -1   -1   0
 $EndComp
 $Comp
 L power:+3.3V #PWR?
 U 1 1 60A70C58
-P 7300 1900
-F 0 "#PWR?" H 7300 1750 50  0001 C CNN
-F 1 "+3.3V" H 7450 2000 50  0000 C CNN
-F 2 "" H 7300 1900 50  0001 C CNN
-F 3 "" H 7300 1900 50  0001 C CNN
-	1    7300 1900
-	1    0    0    -1
-$EndComp
-Wire Wire Line
-	7350 2200 7300 2200
-Wire Wire Line
-	6750 1550 6750 2200
-Connection ~ 7300 2200
-Wire Wire Line
-	7300 2200 6750 2200
+P 7350 2000
+F 0 "#PWR?" H 7350 1850 50  0001 C CNN
+F 1 "+3.3V" H 7500 2100 50  0000 C CNN
+F 2 "" H 7350 2000 50  0001 C CNN
+F 3 "" H 7350 2000 50  0001 C CNN
+	1    7350 2000
+	1    0    0    -1
+$EndComp
 Wire Wire Line
 	6800 1150 7000 1150
 Connection ~ 6800 1150
 Wire Wire Line
-	6750 1550 7000 1550
-Wire Wire Line
 	6950 1450 6950 1250
 Wire Wire Line
@@
 Wire Wire Line
 	6950 1450 7000 1450
+$Comp
+L Device:R R?
+U 1 1 60A04DE5
+P 7800 1900
+F 0 "R?" H 7600 1950 50  0000 L CNN
+F 1 "4K7" V 7800 1850 50  0000 L CNN
+F 2 "Resistor_SMD:R_0603_1608Metric" V 7730 1900 50  0001 C CNN
+F 3 "~" H 7800 1900 50  0001 C CNN
+	1    7800 1900
+	0    -1   -1   0
+$EndComp
+Wire Wire Line
+	7350 2000 7250 2000
+$Comp
+L power:GND #PWR?
+U 1 1 60A47FC5
+P 6600 2100
+F 0 "#PWR?" H 6600 1850 50  0001 C CNN
+F 1 "GND" H 6605 1927 50  0000 C CNN
+F 2 "" H 6600 2100 50  0001 C CNN
+F 3 "" H 6600 2100 50  0001 C CNN
+	1    6600 2100
+	1    0    0    -1
+$EndComp
+Connection ~ 6600 2100
+Wire Wire Line
+	6950 1550 6950 2000
+Wire Wire Line
+	6950 1550 7000 1550
+Wire Wire Line
+	7000 1750 6700 1750
+Wire Wire Line
+	6700 1750 6700 2100
+$Comp
+L Device:D_Zener D?
+U 1 1 60A2F1AD
+P 7650 2050
+F 0 "D?" V 7604 2130 50  0000 L CNN
+F 1 "D_Zener" V 7695 2130 50  0000 L CNN
+F 2 "" H 7650 2050 50  0001 C CNN
+F 3 "~" H 7650 2050 50  0001 C CNN
+	1    7650 2050
+	0    1    1    0
+$EndComp
+Wire Wire Line
+	7650 1900 7500 1900
+Wire Wire Line
+	7500 1900 7500 2100
+Wire Wire Line
+	7500 2100 6950 2100
+Wire Wire Line
+	6950 2100 6950 2000
+Connection ~ 7650 1900
+Connection ~ 6950 2000
+Wire Wire Line
+	6700 2100 6800 2100
+Wire Wire Line
+	6800 2100 6800 2200
+Wire Wire Line
+	6800 2200 7650 2200
+Connection ~ 6700 2100
 $EndSCHEMATC

Commit message: 2021-05-14_02
Parts:
- removed D?: D_Zener, symbol Device:D_Zener
- added D7: BZT52C-3V6, Diode_SMD:D_SOD-123, symbol Device:D_Zener
- added J7: Conn_01x03, Connector2:JST_XH_B3B-XH-AM_1x03_P2.50mm_Vertical, symbol Connector_Generic:Conn_01x03
- added J8: Conn_01x02, Connector2:JST_XH_B2B-XH-AM_1x02_P2.50mm_Vertical, symbol Connector_Generic:Conn_01x02
- D1: value 3V -> BZT52C-3V6; footprint Diode_SMD:D_SMA -> Diode_SMD:D_SOD-123
- J2: footprint Connector2:JST_XH_B2B-XH-AM_1x02_P2.50mm_Vertical -> Connector_JST:JST_XH_B4B-XH-A_1x04_P2.50mm_Vertical
- gave numbers to parts that had none: 4
Connections:
- net +3V3: now also J8.1 (Pin_1)
- net GND: now also D7.2 (A), J8.2 (Pin_2)
- net SCL: now also J7.1 (Pin_1)
- net SDA: now also J7.3 (Pin_3)
- net ~INT: now also J7.2 (Pin_2)
- net at J2.3 (Pin_3), R43.1, R44.1: now also D7.1 (K)
Other:
- note added: "Connectors to Front Panel"
Changed lines of the file:
@@
 F 0 "J2" H 7200 1350 50  0000 C CNN
 F 1 "Conn_01x02" H 7350 1750 50  0001 C CNN
-F 2 "Connector2:JST_XH_B2B-XH-AM_1x02_P2.50mm_Vertical" H 7200 1650 50  0001 C CNN
+F 2 "Connector_JST:JST_XH_B4B-XH-A_1x04_P2.50mm_Vertical" H 7200 1650 50  0001 C CNN
 F 3 "~" H 7200 1650 50  0001 C CNN
 	1    7200 1650
@@
 P 1100 3750
 F 0 "D1" V 1000 3750 50  0000 L CNN
-F 1 "3V" V 1200 3750 50  0000 L CNN
-F 2 "Diode_SMD:D_SMA" H 1100 3750 50  0001 C CNN
+F 1 "BZT52C-3V6" V 1300 3650 50  0000 L CNN
+F 2 "Diode_SMD:D_SOD-123" H 1100 3750 50  0001 C CNN
 F 3 "~" H 1100 3750 50  0001 C CNN
 	1    1100 3750
@@
 	6600 2100 6700 2100
 $Comp
-L Device:Q_NMOS_GSD Q?
+L Device:Q_NMOS_GSD Q6
 U 1 1 609EE83B
 P 3200 3650
-F 0 "Q?" H 3404 3696 50  0000 L CNN
-F 1 "Si2306" H 3150 3900 50  0000 L CNN
+F 0 "Q6" H 3404 3696 50  0000 L CNN
+F 1 "Si2306" H 3000 3500 50  0000 L CNN
 F 2 "Package_TO_SOT_SMD:SOT-23" H 3400 3750 50  0001 C CNN
 F 3 "~" H 3200 3650 50  0001 C CNN
@@
 	1750 4300 3800 4300
 $Comp
-L Connector_Generic:Conn_01x02 J?
+L Connector_Generic:Conn_01x02 J10
 U 1 1 60A56CFA
 P 7200 1150
-AR Path="/60A56CFA" Ref="J?"  Part="1"
+AR Path="/60A56CFA" Ref="J10"  Part="1"
 AR Path="/60357CC4/60A56CFA" Ref="J?"  Part="1"
-F 0 "J?" H 7400 1100 50  0000 C CNN
-F 1 "Conn_01x02" H 7118 1276 50  0000 C CNN
+F 0 "J10" H 7200 1250 50  0000 C CNN
+F 1 "Conn_01x02" H 7118 1276 50  0001 C CNN
 F 2 "Connector2:JST_XH_B2B-XH-AM_1x02_P2.50mm_Vertical" H 7200 1150 50  0001 C CNN
 F 3 "~" H 7200 1150 50  0001 C CNN
@@
 $EndComp
 $Comp
-L Device:R R?
+L Device:R R43
 U 1 1 60A70C52
 P 7100 2000
-F 0 "R?" V 7200 2050 50  0000 L CNN
+F 0 "R43" V 7200 2050 50  0000 L CNN
 F 1 "10K" V 7100 1950 50  0000 L CNN
 F 2 "Resistor_SMD:R_0603_1608Metric" V 7030 2000 50  0001 C CNN
@@
 $EndComp
 $Comp
-L power:+3.3V #PWR?
+L power:+3.3V #PWR0101
 U 1 1 60A70C58
 P 7350 2000
-F 0 "#PWR?" H 7350 1850 50  0001 C CNN
-F 1 "+3.3V" H 7500 2100 50  0000 C CNN
+F 0 "#PWR0101" H 7350 1850 50  0001 C CNN
+F 1 "+3.3V" H 7350 2150 50  0000 C CNN
 F 2 "" H 7350 2000 50  0001 C CNN
 F 3 "" H 7350 2000 50  0001 C CNN
@@
 	6950 1450 7000 1450
 $Comp
-L Device:R R?
+L Device:R R44
 U 1 1 60A04DE5
 P 7800 1900
-F 0 "R?" H 7600 1950 50  0000 L CNN
+F 0 "R44" V 7650 1950 50  0000 L CNN
 F 1 "4K7" V 7800 1850 50  0000 L CNN
 F 2 "Resistor_SMD:R_0603_1608Metric" V 7730 1900 50  0001 C CNN
@@
 	7350 2000 7250 2000
 $Comp
-L power:GND #PWR?
+L power:GND #PWR0102
 U 1 1 60A47FC5
 P 6600 2100
-F 0 "#PWR?" H 6600 1850 50  0001 C CNN
+F 0 "#PWR0102" H 6600 1850 50  0001 C CNN
 F 1 "GND" H 6605 1927 50  0000 C CNN
 F 2 "" H 6600 2100 50  0001 C CNN
@@
 Wire Wire Line
 	6700 1750 6700 2100
-$Comp
-L Device:D_Zener D?
-U 1 1 60A2F1AD
-P 7650 2050
-F 0 "D?" V 7604 2130 50  0000 L CNN
-F 1 "D_Zener" V 7695 2130 50  0000 L CNN
-F 2 "" H 7650 2050 50  0001 C CNN
-F 3 "~" H 7650 2050 50  0001 C CNN
-	1    7650 2050
+Wire Wire Line
+	7650 1900 7600 1900
+Wire Wire Line
+	7500 1900 7500 2100
+Wire Wire Line
+	7500 2100 6950 2100
+Wire Wire Line
+	6950 2100 6950 2000
+Connection ~ 6950 2000
+Wire Wire Line
+	6700 2100 6800 2100
+Wire Wire Line
+	6800 2100 6800 2200
+Wire Wire Line
+	6800 2200 7600 2200
+Connection ~ 6700 2100
+Text Notes 7300 1250 0    50   ~ 0
+GND
+Text Notes 7300 1150 0    50   ~ 0
+PWM
+$Comp
+L Device:D_Zener D7
+U 1 1 609FA542
+P 7600 2050
+F 0 "D7" V 7700 1900 50  0000 L CNN
+F 1 "BZT52C-3V6" V 7700 2050 50  0000 L CNN
+F 2 "Diode_SMD:D_SOD-123" H 7600 2050 50  0001 C CNN
+F 3 "~" H 7600 2050 50  0001 C CNN
+	1    7600 2050
 	0    1    1    0
 $EndComp
-Wire Wire Line
-	7650 1900 7500 1900
-Wire Wire Line
-	7500 1900 7500 2100
-Wire Wire Line
-	7500 2100 6950 2100
-Wire Wire Line
-	6950 2100 6950 2000
-Connection ~ 7650 1900
-Connection ~ 6950 2000
-Wire Wire Line
-	6700 2100 6800 2100
-Wire Wire Line
-	6800 2100 6800 2200
-Wire Wire Line
-	6800 2200 7650 2200
-Connection ~ 6700 2100
+Connection ~ 7600 1900
+Wire Wire Line
+	7600 1900 7500 1900
+Wire Notes Line
+	6850 6650 5400 6650
+$Comp
+L Connector_Generic:Conn_01x03 J7
+U 1 1 60A1B349
+P 5800 5800
+AR Path="/60A1B349" Ref="J7"  Part="1"
+AR Path="/60357CC4/60A1B349" Ref="J?"  Part="1"
+F 0 "J7" H 6000 5800 50  0000 C CNN
+F 1 "Conn_01x03" H 5718 6026 50  0000 C CNN
+F 2 "Connector2:JST_XH_B3B-XH-AM_1x03_P2.50mm_Vertical" H 5800 5800 50  0001 C CNN
+F 3 "~" H 5800 5800 50  0001 C CNN
+	1    5800 5800
+	-1   0    0    -1
+$EndComp
+$Comp
+L Connector_Generic:Conn_01x02 J8
+U 1 1 60A1B34F
+P 5800 6250
+AR Path="/60A1B34F" Ref="J8"  Part="1"
+AR Path="/60357CC4/60A1B34F" Ref="J?"  Part="1"
+F 0 "J8" H 6000 6200 50  0000 C CNN
+F 1 "Conn_01x02" H 5718 6376 50  0000 C CNN
+F 2 "Connector2:JST_XH_B2B-XH-AM_1x02_P2.50mm_Vertical" H 5800 6250 50  0001 C CNN
+F 3 "~" H 5800 6250 50  0001 C CNN
+	1    5800 6250
+	-1   0    0    -1
+$EndComp
+Wire Wire Line
+	6000 6250 6250 6250
+Wire Wire Line
+	6000 6350 6250 6350
+Wire Wire Line
+	6000 5700 6200 5700
+Wire Wire Line
+	6000 5900 6200 5900
+Wire Wire Line
+	6000 5800 6450 5800
+Text GLabel 6200 5700 2    50   Input ~ 0
+SCL
+Text GLabel 6200 5900 2    50   Input ~ 0
+SDA
+$Comp
+L power:+3.3V #PWR0104
+U 1 1 60A1B35C
+P 6250 6250
+AR Path="/60A1B35C" Ref="#PWR0104"  Part="1"
+AR Path="/60357CC4/60A1B35C" Ref="#PWR?"  Part="1"
+F 0 "#PWR0104" H 6250 6100 50  0001 C CNN
+F 1 "+3.3V" H 6265 6423 50  0000 C CNN
+F 2 "" H 6250 6250 50  0001 C CNN
+F 3 "" H 6250 6250 50  0001 C CNN
+	1    6250 6250
+	1    0    0    -1
+$EndComp
+Wire Notes Line
+	5400 5400 6850 5400
+Wire Notes Line
+	6850 5400 6850 6650
+Wire Notes Line
+	5400 6650 5400 5400
+Text Notes 5450 5500 0    50   ~ 0
+Connectors to Front Panel
+Text GLabel 6450 5800 2    50   Input ~ 0
+~INT
+$Comp
+L power:GND #PWR?
+U 1 1 60A1B367
+P 6250 6350
+AR Path="/60357CC4/60A1B367" Ref="#PWR?"  Part="1"
+AR Path="/60A1B367" Ref="#PWR0105"  Part="1"
+F 0 "#PWR0105" H 6250 6100 50  0001 C CNN
+F 1 "GND" H 6255 6177 50  0000 C CNN
+F 2 "" H 6250 6350 50  0001 C CNN
+F 3 "" H 6250 6350 50  0001 C CNN
+	1    6250 6350
+	1    0    0    -1
+$EndComp
 $EndSCHEMATC
