File: NieuwOntwerp/Load.sch (KiCad schematic (older format))
At the start: 85 parts, among them J1 USB_C_Receptacle_USB2.0, J10 Conn_01x02, J2 Conn_01x02, J7 Conn_01x03, J8 Conn_01x02, Q1 Si2306, Q2 4809NG, Q3 IRF840, Q4 IRF840, Q5 IRF840, Q6 Si2306, U1 ESP12E, U2 FT231XQ, U3 LM358, U4 MCP4725A0, U5 LM358, U6 

Commit message: 2021-05-15_02
Connections:
- net +12V: no longer R18.2
- net +5V: now also R18.2
Changed lines of the file:
@@
 Connection ~ 6400 3700
-$Comp
-L power:+12V #PWR023
-U 1 1 607E4EF7
-P 6400 3400
-F 0 "#PWR023" H 6400 3250 50  0001 C CNN
-F 1 "+12V" H 6550 3500 50  0000 C CNN
-F 2 "" H 6400 3400 50  0001 C CNN
-F 3 "" H 6400 3400 50  0001 C CNN
-	1    6400 3400
-	1    0    0    -1
-$EndComp
 $Comp
 L Device:R R26
@@
 	1    0    0    -1
 $EndComp
+$Comp
+L power:+5V #PWR?
+U 1 1 60A58FD8
+P 6400 3400
+F 0 "#PWR?" H 6400 3250 50  0001 C CNN
+F 1 "+5V" H 6500 3500 50  0000 C CNN
+F 2 "" H 6400 3400 50  0001 C CNN
+F 3 "" H 6400 3400 50  0001 C CNN
+	1    6400 3400
+	1    0    0    -1
+$EndComp

Commit message: 2021-05-16_01
Changed lines of the file:
@@
 	3150 1450 3700 1450
 Connection ~ 3700 1450
-Wire Wire Line
-	1200 900  1350 900
 $Comp
 L Device:R R1
@@
 Wire Wire Line
 	1350 1150 1350 900
-Connection ~ 1350 900
 Wire Wire Line
 	1300 1900 1300 1750
