File: NieuwOntwerp/Load.sch (KiCad schematic (older format))
At the start: 85 parts, among them J1 USB_C_Receptacle_USB2.0, J10 Conn_01x02, J2 Conn_01x02, J7 Conn_01x03, J8 Conn_01x02, Q1 Si2306, Q2 4809NG, Q3 IRF840, Q4 IRF840, Q5 IRF840, Q6 Si2306, U1 ESP12E, U2 FT231XQ, U3 LM358, U4 MCP4725A0, U5 LM358, U6 

Commit message: start
Parts:
- removed R24: 1K, Resistor_SMD:R_0603_1608Metric, symbol Device:R
- added D10, D9: MMSZ5225/3V, Diode_SMD:D_SOD-123, symbol Device:D_Zener
- added R? (x2): 10K, Resistor_SMD:R_0603_1608Metric, symbol Device:R
- added R?: 27K, Resistor_SMD:R_0603_1608Metric, symbol Device:R
- added R?: 1K, Resistor_SMD:R_0603_1608Metric, symbol Device:R
- C5: value 100uF -> 47uF; footprint Capacitor_THT:CP_Radial_D6.3mm_P2.50mm -> Capacitor_THT:CP_Radial_D5.0mm_P2.00mm
- C6: value 470pF -> 4,7nF
- R20: value 100K -> 4K7
- RV1: footprint Potentiometer_THT:Potentiometer_Bourns_3266Y_Vertical -> Potentiometer_THT:Potentiometer_Bourns_3296W_Vertical
- U6: value (none) -> INA219; footprint Package_SO:SOIC-8_3.9x4.9mm_P1.27mm -> Package_TO_SOT_SMD:SOT-23-8
Connections:
- net +12V: now also R10.2, RV1.2
- net +3V3: now also R?.2
- net +5V: no longer R10.2, RV1.2
- net GND: now also C6.1, R11.1, D10.2 (A), D9.2 (A), R?.1, R?.1; no longer H2.1
- net RTS: now also R?.1
- net THERM: now also R?.2
- net at U1.10 (GPIO15): now also R?.2
- net at R5.1, U2.8 (USBDP): now also D9.1 (K)
- net at R4.1, U2.9 (USBDM): now also D10.1 (K)
- net at Q2.1 (G), R20.2, U3.7: now also R?.2
- net at D6.2 (A), J10.2 (Pin_2), Q2.2 (D): no longer J2.4 (Pin_4)
- new net: J2.4 (Pin_4), R?.1
- no-connect marks 18 -> 19
Other:
- note added: "4V"
- note added: "700Ohm = 120gr\n2KOhm = 20gr"
- note added: "8V"
- note added: "900 Ohm = minimale snelheid = 8V"
- note added: "Connector te dicht tegen de andere"
- moved on the sheet: D6, D7, H2, H4, J10, Q2, R20, R43, R44
