File: NieuwOntwerp/Load.sch (KiCad schematic (older format))
At the start: 86 parts, among them J1 USB_C_Receptacle_USB2.0, J10 Conn_01x02, J2 Conn_01x02, J7 Conn_01x03, J8 Conn_01x02, Q2 4809NG, Q3 IRF840, Q4 IRF840, Q5 IRF840, Q6 Si2306, U1 ESP12E, U2 FT231XQ, U3 LM358, U4 MCP4725A0, U5 LM358, U6 INA219

Commit message: MCP4725 BEGIN
Other:
- note added: "Fan start/stop"
- note removed: "Fan start"
Changed lines of the file:
@@
 	1750 4300 1750 2850
 Text Notes 1800 2950 0    50   ~ 0
-Fan start
+Fan start/stop
 $Comp
 L Device:Q_NMOS_GSD Q6

Commit message: Print_update
Parts:
- removed D1: BZT52C-3V6, Diode_SMD:D_SOD-123, symbol Device:D_Zener
- removed D10, D9: MMSZ5225/3V, Diode_SMD:D_SOD-123, symbol Device:D_Zener
- removed J7: Conn_01x03, Connector2:JST_XH_B3B-XH-AM_1x03_P2.50mm_Vertical, symbol Connector_Generic:Conn_01x03
- removed J8: Conn_01x02, Connector2:JST_XH_B2B-XH-AM_1x02_P2.50mm_Vertical, symbol Connector_Generic:Conn_01x02
- removed R1: 330K, Resistor_SMD:R_0603_1608Metric, symbol Device:R
- removed R2: 10k, Resistor_SMD:R_0603_1608Metric, symbol Device:R
- added J7: Din_02x03, Connector_IDC:IDC-Header_2x03_P2.54mm_Vertical, symbol Connector_Generic:Conn_02x03_Odd_Even
- C1, C3: footprint Capacitor_SMD:C_0603_1608Metric -> Capacitor_SMD:C_0402_1005Metric
- R4, R5: footprint Resistor_SMD:R_0603_1608Metric -> Resistor_SMD:R_0402_1005Metric
- gave numbers to parts that had none: 5
Connections:
- net +5V is gone; now on net +12V: R18.2
- net +3V3: now also J7.4 (Pin_4)
- net GND: now also R28.1, R32.1, R37.1, J7.6 (Pin_6); no longer H1.1, R31.1, R34.2
- net LOAD: now also R31.2, R33.2; no longer Q3.2 (D), Q4.2 (D), Q5.2 (D)
- net SCL: now also J7.3 (Pin_3)
- net SDA: now also J7.1 (Pin_1)
- net SHUNT: now also Q3.2 (D), Q4.2 (D), Q5.2 (D), R31.1, R34.2; no longer R28.1, R31.2, R32.1, R33.2, R37.1
- net ~INT: now also J7.5 (Pin_5)
- net Earth: now reaches H2.1
- net Earth: now also H1.1
- net ADC: no longer names the net of U1.2 (ADC)
- no-connect marks 19 -> 20
Other:
- note removed: "4V"
- note removed: "700Ohm = 120gr\n2KOhm = 20gr"
- note removed: "8V"
- note removed: "900 Ohm = minimale snelheid = 8V"
- note removed: "VOLT Measure"
- moved on the sheet: H2, H4

Commit message: print update
Connections:
- net at R21.1, R22.2: now also U5.3 (+); no longer U5.5 (+)
- net at R23.2, R25.2: now also U5.2 (-); no longer U5.6 (-)
- net at R25.1, R26.1, R29.1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: now also U5.1; no longer U5.7
- net at U4.1 (VOUT): now also U5.5 (+); no longer U5.3 (+)
- net at R17.1, R21.2: now also U5.7; no longer U5.1
- net at R16.2, R17.2: now also U5.6 (-); no longer U5.2 (-)
Changed lines of the file:
@@
 $Comp
 L Amplifier_Operational:LM358 U5
-U 2 1 6011E1C0
+U 1 1 6011E1C0
 P 7000 3800
 F 0 "U5" H 6950 3800 50  0000 C CNN
@@
 F 2 "Package_SO:SOIC-8_3.9x4.9mm_P1.27mm" H 7000 3800 50  0001 C CNN
 F 3 "http://www.ti.com/lit/ds/symlink/lm2904-n.pdf" H 7000 3800 50  0001 C CNN
-	2    7000 3800
+	1    7000 3800
 	1    0    0    -1
 $EndComp
@@
 $Comp
 L Amplifier_Operational:LM358 U5
-U 1 1 6076B910
+U 2 1 6076B910
 P 6100 3000
 F 0 "U5" H 6050 3000 50  0000 C CNN
@@
 F 2 "Package_SO:SOIC-8_3.9x4.9mm_P1.27mm" H 6100 3000 50  0001 C CNN
 F 3 "http://www.ti.com/lit/ds/symlink/lm2904-n.pdf" H 6100 3000 50  0001 C CNN
-	1    6100 3000
-	1    0    0    -1
-$EndComp
+	2    6100 3000
+	1    0    0    -1
+$EndComp

Commit message: 21-11-2021
Parts:
- removed U6: INA219, Package_TO_SOT_SMD:SOT-23-8, symbol Analog_ADC:INA219AxD
- added U6: INA219AxDCN, Package_TO_SOT_SMD:SOT-23-8, symbol Analog_ADC:INA219AxDCN
Connections:
- net +3V3: now also U6.4 (VS)
- net GND: now also U6.3 (GND), U6.7 (A0), U6.8 (A1)
- net SCL: now also U6.5 (SCL)
- net SDA: now also U6.6 (SDA)
- net at C9.2, R34.1: now also U6.2 (IN-)
- net at C9.1, R33.1: now also U6.1 (IN+)
Changed lines of the file:
@@
 $EndDescr
-$Comp
-L Analog_ADC:INA219AxD U6
-U 1 1 60103786
-P 10350 1500
-F 0 "U6" H 10350 1500 50  0000 C CNN
-F 1 "INA219" H 10550 1900 50  0000 C CNN
-F 2 "Package_TO_SOT_SMD:SOT-23-8" H 11150 1150 50  0001 C CNN
-F 3 "https://www.ti.com/lit/ds/symlink/ina219.pdf" H 10700 1400 50  0001 C CNN
-	1    10350 1500
-	1    0    0    -1
-$EndComp
 $Comp
 L Device:C C9
@@
 	6400 7450 6550 7450
 $Comp
-L power:GND #PWR?
+L power:GND #PWR0114
 U 1 1 616961E5
 P 6550 7450
-F 0 "#PWR?" H 6550 7200 50  0001 C CNN
+F 0 "#PWR0114" H 6550 7200 50  0001 C CNN
 F 1 "GND" H 6450 7350 50  0000 C CNN
 F 2 "" H 6550 7450 50  0001 C CNN
@@
 Wire Wire Line
 	2600 6350 2750 6350
+$Comp
+L Analog_ADC:INA219AxDCN U6
+U 1 1 6199056C
+P 10350 1500
+F 0 "U6" H 10350 2081 50  0000 C CNN
+F 1 "INA219AxDCN" H 10650 1900 50  0000 C CNN
+F 2 "Package_TO_SOT_SMD:SOT-23-8" H 11000 1150 50  0001 C CNN
+F 3 "http://www.ti.com/lit/ds/symlink/ina219.pdf" H 10700 1400 50  0001 C CNN
+	1    10350 1500
+	1    0    0    -1
+$EndComp
 $EndSCHEMATC
