File: NieuwOntwerp/Load.kicad_pcb (KiCad board)
At the start: 2 copper layers, 84 x 96 mm, 104 parts, among them J1 Conn_01x02, J2 Conn_01x02, J3 Conn_01x05, J4 Conn_01x03, J5 Conn_01x02, J6 Conn_01x03, J7 Conn_01x02, Q1 IRF840, Q2 IRF840, SW1 Switch_6x6_SMT, SW2 Switch_6x6_SMT, SW3 Switch_6x6_SMT, SW4 Switch_6x6_SMT, T1 EE13, U1 ESP12E, U10 MCP4725A0, U2 LNK364D, U3 LM358, U4 PC817, U5 TL431, U6 LM1117-3.3, U7 LM358, U8 SSD1306, U9 PCF8574

Commit message: Sync_21-04-27
Parts:
- removed REF** (x3): DOUBLE_SIDED_TAB, Panellizing:DOUBLE_SIDED_TAB
- added C23: 10nF, Capacitor_SMD:C_0603_1608Metric, F.Cu at (60.0, 57.0)
- added C24: X type 470pF, Capacitor_SMD:C_0603_1608Metric, F.Cu at (36.6, 45.7)
- added C25: 100n, Capacitor_SMD:C_0603_1608Metric, F.Cu at (66.7, 51.2)
- added C26: 100n, Capacitor_SMD:C_0603_1608Metric, F.Cu at (52.2, 63.4)
- added C27: 100n, Capacitor_SMD:C_0603_1608Metric, F.Cu at (56.2, 60.9)
- added C28: 100n, Capacitor_SMD:C_0603_1608Metric, F.Cu at (52.2, 60.9)
- added C29: 100nF, Capacitor_SMD:C_0603_1608Metric, F.Cu at (74.1, 42.8)
- added C30: 4,7uF, Capacitor_SMD:C_Elec_4x5.4, F.Cu at (56.5, 50.3)
- added D10: SS34, Diode_SMD:D_SMA, F.Cu at (61.9, 41.8)
- added D11: LED, LED_SMD:LED_0603_1608Metric, F.Cu at (103.3, 34.6)
- added D9: FR107, Diode_SMD:D_SMA, F.Cu at (48.3, 56.1)
- added FB1: 1K, Resistor_SMD:R_0603_1608Metric, F.Cu at (106.2, 37.1)
- added J8: Conn_01x02, Connector2:JST_XH_B3B-XH-AM_1x03_P2.50mm_Vertical, F.Cu at (30.2, 40.0)
- added Q3: P3057G, Package_TO_SOT_SMD:SOT-89-3, F.Cu at (69.0, 42.5)
- added R17: 8k6, Resistor_SMD:R_1210_3225Metric, F.Cu at (43.4, 65.1)
- added R33: 18R, Resistor_SMD:R_1206_3216Metric, F.Cu at (63.1, 45.8)
- added R34: 150, Resistor_SMD:R_0603_1608Metric, F.Cu at (54.3, 58.4)
- added R35: 1K, Resistor_SMD:R_0603_1608Metric, F.Cu at (48.2, 63.8)
- added R36: 22k, Resistor_SMD:R_0402_1005Metric, F.Cu at (47.6, 66.1)
- added R37: 6K8, Resistor_SMD:R_0603_1608Metric, F.Cu at (64.0, 53.7)
- added R38: 27R, Resistor_SMD:R_0603_1608Metric, F.Cu at (96.6, 43.6)
- added R39: 27R, Resistor_SMD:R_0603_1608Metric, F.Cu at (102.2, 37.7)
- added R40: 1K6, Resistor_SMD:R_0603_1608Metric, F.Cu at (107.3, 34.6)
- added R41: 1K6, Resistor_SMD:R_0603_1608Metric, F.Cu at (100.6, 41.0)
- added R6: 0R002, Resistor_SMD:R_1206_3216Metric, F.Cu at (104.0, 31.7)
- added U11: TL431, Package_TO_SOT_SMD:SOT-23, F.Cu at (62.5, 49.7)
- added U12: LM1117-3.3, Package_TO_SOT_SMD:SOT-223-3_TabPin2, F.Cu at (15.7, 63.0)
- added U13: FT231XQ, Package_DFN_QFN:QFN-20-1EP_4x4mm_P0.5mm_EP2.5x2.5mm, F.Cu at (91.5, 42.7)
- C1: value X2 100nF/275V -> Y type 2N2/250VAC; footprint Condensator:CBB22104J400V -> Condensator:JN_102M
- C10: value 100n -> 10n; footprint Capacitor_SMD:C_0603_1608Metric -> Capacitor_SMD:C_0402_1005Metric
- C11: value 100n -> 6,8uF/400V; footprint Capacitor_SMD:C_0603_1608Metric -> Capacitor_THT:CP_Radial_D8.0mm_P3.50mm
- C12: value 100nF -> 1nF/300V; footprint Capacitor_SMD:C_0603_1608Metric -> Condensator:JN_102M
- C13: value 100uF/25V -> 100nF/50V; footprint Capacitor_THT:CP_Radial_D5.0mm_P2.00mm -> Capacitor_SMD:C_0603_1608Metric
- C14: value 100n -> 1000uF/25V; footprint Capacitor_SMD:C_0603_1608Metric -> Capacitor_THT:CP_Radial_D10.0mm_P5.00mm
- C15: value 10nF -> 470pF/50V
- C16: value 100n -> 100nF
- C17: value X type 470pF -> 100uF/25V; footprint Capacitor_SMD:C_0603_1608Metric -> Capacitor_THT:CP_Radial_D5.0mm_P2.00mm
- C2: value 4,7uF/400V -> 47pF; footprint Capacitor_THT:CP_Radial_D8.0mm_P3.50mm -> Capacitor_SMD:C_0603_1608Metric
- C3: value 6,8uF/400V -> 10nF; footprint Capacitor_THT:CP_Radial_D8.0mm_P3.50mm -> Capacitor_SMD:C_0402_1005Metric
- C4: value 1nF/300V -> Y type 2N2/250VAC
- C5: value Y type 2N2/250VAC -> 47pF; footprint Condensator:JN_102M -> Capacitor_SMD:C_0603_1608Metric
- C6: value 100nF/50V -> 100nF
- C7: value Y type 2N2/250VAC -> X2 100nF/275V; footprint Condensator:JN_102M -> Condensator:CBB22104J400V
- C8: value 1000uF/25V -> 470uF/16V; footprint Capacitor_THT:CP_Radial_D10.0mm_P5.00mm -> Capacitor_THT:CP_Radial_D8.0mm_P3.80mm
- C9: value 470pF/50V -> 4,7uF/400V; footprint Capacitor_SMD:C_0603_1608Metric -> Capacitor_THT:CP_Radial_D8.0mm_P3.50mm
- D2: value DB207S -> LED; footprint Diode2:SOT4_Rectifier_Bridge -> LED_SMD:LED_0603_1608Metric
- D3: value FR107 -> DB207S; footprint Diode_SMD:D_SMA -> Diode2:SOT4_Rectifier_Bridge
- D4: value SS34 -> US1K
- J1: value Conn_01x02 -> USB_C_Receptacle_USB2.0; footprint Connector2:JST_XH_B3B-XH-AM_1x03_P2.50mm_Vertical -> Connector2:USB-C_Receptable_SMD_16pin
- J3: value Conn_01x05 -> Conn_01x02; footprint Connector2:Molex_PicoBlade_53047-0510_1x05_P1.25mm_Vertical -> Connector2:JST_XH_B2B-XH-AM_1x02_P2.50mm_Vertical
- Q1: value IRF840 -> 4809NG
- R1, R16, R19, R2, R22, R23, R24, R25, R26, R27, R28, R29, R3, R30, R31, R32: footprint Resistor_SMD:R_0603_1608Metric_Pad1.05x0.95mm_HandSolder -> Resistor_SMD:R_0603_1608Metric
- R11: value 18R -> 6K8; footprint Resistor_SMD:R_1206_3216Metric -> Resistor_SMD:R_0603_1608Metric
- R12: value 150 -> 10K
- R13: value 1K -> 150R
- R14: value 22k -> 100K; footprint Resistor_SMD:R_0402_1005Metric -> Resistor_SMD:R_0603_1608Metric
- R15: value 6K8 -> 300R; footprint Resistor_SMD:R_0603_1608Metric -> Resistor_SMD:R_1210_3225Metric
- R5: value 10R -> 0R002; footprint Resistor_SMD:R_2512_6332Metric -> Resistor_SMD:R_1206_3216Metric
- R7: value 300R -> 10R; footprint Resistor_SMD:R_1210_3225Metric -> Resistor_SMD:R_2512_6332Metric
- R8: value 100k -> 10K; footprint Resistor_SMD:R_1210_3225Metric -> Resistor_SMD:R_0603_1608Metric
- U2: value LNK364D -> LM358; footprint Package_SO:PowerIntegrations_SO-8C -> Package_SO:SOIC-8_3.9x4.9mm_P1.27mm
- U4: value PC817 -> MCP4725A0; footprint Package_SO:SSO-4_6.7x5.1mm_P2.54mm_Clearance8mm -> Package_TO_SOT_SMD:SOT-23-6
- U5: value TL431 -> LNK364D; footprint Package_TO_SOT_SMD:SOT-23 -> Package_SO:PowerIntegrations_SO-8C
- U6: value LM1117-3.3 -> PC817; footprint Package_TO_SOT_SMD:SOT-223-3_TabPin2 -> Package_SO:SSO-4_6.7x5.1mm_P2.54mm_Clearance8mm
- moved C11 130.9 mm to (28.1, 49.2)
- moved C14 121.0 mm to (26.6, 60.0)
- moved J5 111.8 mm to (38.3, 58.5)
- moved RV1 109.3 mm to (16.9, 56.5)
- moved C9 108.5 mm to (41.9, 42.6)
- moved R15 108.5 mm to (47.1, 60.5)
- moved C12 108.4 mm to (37.7, 83.9)
- moved R11 106.2 mm to (53.7, 80.5)
- moved U6 103.0 mm to (33.2, 33.3)
- moved L1 99.8 mm to (18.7, 35.7)
- moved F1 99.2 mm to (55.1, 55.5)
- moved J2 97.1 mm to (38.3, 50.7)
- moved U5 96.5 mm to (48.5, 50.6)
- moved R7 93.1 mm to (65.8, 32.5)
- moved C17 92.6 mm to (72.5, 33.3)
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Connections:
- C1 pad 1: Net-(C1-Pad1) -> Earth
- C1 pad 2: NEUTRAL -> Net-(C1-Pad2)
- C10 pad 1: GND -> GNDA
- C10 pad 2: +3V3 -> Net-(C10-Pad2)
- C11 pad 1: GND -> Net-(C11-Pad1)
- C11 pad 2: +3V3 -> Net-(C11-Pad2)
- C12 pad 1: Net-(C12-Pad1) -> Net-(C11-Pad1)
- C13 pad 1: +10V -> Net-(C13-Pad1)
- C13 pad 2: Net-(C13-Pad2) -> Net-(C11-Pad2)
- C14 pad 1: GND -> Net-(C14-Pad1)
- C14 pad 2: +3V3 -> GND
- C15 pad 1: +10V -> Net-(C14-Pad1)
- C15 pad 2: GND -> Net-(C15-Pad2)
- C16 pad 1: GND -> Net-(C16-Pad1)
- C16 pad 2: +3V3 -> Net-(C16-Pad2)
- C17 pad 1: Earth -> +12V
- C2 pad 2: Net-(C2-Pad2) -> GND
- C3 pad 2: Net-(C3-Pad2) -> GND
- C4 pad 1: Net-(C3-Pad1) -> NEUTRAL
- C4 pad 2: Net-(C4-Pad2) -> Earth
- C5 pad 1: Earth -> Net-(C5-Pad1)
- C5 pad 2: Net-(C5-Pad2) -> GND
- C6 pad 2: Net-(C3-Pad2) -> GND
- C7 pad 1: NEUTRAL -> Net-(C7-Pad1)
- C7 pad 2: Earth -> NEUTRAL
- C8 pad 2: Net-(C8-Pad2) -> GNDA
- C9 pad 1: Net-(C8-Pad1) -> Net-(C9-Pad1)
- D2 pad 1: NEUTRAL -> Net-(D2-Pad1)
- D2 pad 2: Net-(C1-Pad1) -> Net-(D2-Pad2)
- D3 pad 1: Net-(D3-Pad1) -> NEUTRAL
- D3 pad 2: Net-(D3-Pad2) -> Net-(C7-Pad1)
- D4 pad 2: Net-(D4-Pad2) -> GNDA
- F1 pad 1: Net-(C5-Pad2) -> Net-(C1-Pad2)
- J2 pad 1: LOAD -> Net-(C8-Pad1)
- J2 pad 2: GND -> GNDA
- J3 pad 1: Net-(J3-Pad1) -> LOAD
- J3 pad 2: Net-(J3-Pad2) -> GND
- J6 pad 1: /Front/SCL -> SCL
- J6 pad 3: /Front/SDA -> SDA
- L1 pad 1: Net-(C2-Pad1) -> Net-(C9-Pad1)
- L1 pad 2: Net-(C2-Pad2) -> Net-(C9-Pad2)
- L1 pad 3: Net-(C3-Pad2) -> Net-(C11-Pad2)
- L1 pad 4: Net-(C3-Pad1) -> Net-(C11-Pad1)
- L2 pad 1: Net-(C8-Pad1) -> Net-(C14-Pad1)
- L2 pad 2: +10V -> +12V
- Q1 pad 3: SHUNT -> Net-(Q1-Pad3)
- Q2 pad 3: SHUNT -> Net-(Q2-Pad3)
- R11 pad 1: Net-(C9-Pad2) -> GNDA
- R11 pad 2: Net-(D4-Pad2) -> Net-(R11-Pad2)
- R12 pad 1: Net-(R12-Pad1) -> Net-(C8-Pad1)
- R12 pad 2: Net-(C8-Pad1) -> Net-(R11-Pad2)
- R13 pad 1: Net-(R12-Pad1) -> Net-(Q3-Pad1)
- R13 pad 2: Net-(C12-Pad1) -> Net-(C10-Pad2)
- R14 pad 1: +10V -> Net-(C8-Pad1)
- R14 pad 2: Net-(C12-Pad2) -> Net-(Q3-Pad1)
- R15 pad 2: GND -> Net-(D9-Pad1)
- R19 pad 2: SHUNT -> Net-(Q1-Pad3)
- R2 pad 2: /RTS -> RTS
- R23 pad 2: SHUNT -> Net-(Q2-Pad3)
- R5 pad 1: Net-(C1-Pad1) -> SHUNT
- R5 pad 2: Net-(C5-Pad2) -> Net-(Q1-Pad3)
- R7 pad 1: Net-(C4-Pad2) -> Net-(C7-Pad1)
- R7 pad 2: Net-(D3-Pad1) -> Net-(C1-Pad2)
- R8 pad 1: Net-(C3-Pad1) -> GNDA
- R8 pad 2: Net-(C4-Pad2) -> Net-(R8-Pad2)
- RV1 pad 1: Net-(C5-Pad2) -> Net-(C1-Pad2)
- T1 pad 1: Net-(C3-Pad1) -> Net-(C11-Pad1)
- T1 pad 2: Net-(D3-Pad2) -> Net-(D9-Pad2)
- T1 pad 4: Net-(D4-Pad2) -> Net-(D10-Pad2)
- U1 pad 12: /DTR -> DTR
- U1 pad 15: Net-(J3-Pad2) -> RX
- U1 pad 16: Net-(J3-Pad1) -> TX
- U1 pad 3: /RTS -> RTS
- U2 pad 1: Net-(C6-Pad1) -> Net-(U2-Pad1)
- U2 pad 4: Net-(D3-Pad2) -> GND
- U2 pad 5: Net-(C3-Pad2) -> (no net)
- U2 pad 6: Net-(C3-Pad2) -> (no net)
- U2 pad 7: Net-(C3-Pad2) -> (no net)
- U2 pad 8: Net-(C3-Pad2) -> +12V
- U3 pad 4: GND -> (no net)
- U3 pad 5: (no net) -> Net-(R8-Pad2)
- U3 pad 6: (no net) -> Net-(R11-Pad2)
- U3 pad 7: (no net) -> Net-(C10-Pad2)
- U3 pad 8: +10V -> (no net)
- U4 pad 1: Net-(R12-Pad1) -> Net-(R8-Pad2)
- U4 pad 2: Net-(C12-Pad1) -> GNDA
- U4 pad 3: Net-(U2-Pad2) -> +3V3
- U4 pad 4: Net-(C6-Pad1) -> SDA
- U5 pad 1: Net-(C12-Pad1) -> Net-(C13-Pad1)
- U5 pad 2: Net-(C12-Pad2) -> Net-(U5-Pad2)
- U6 pad 1: GND -> Net-(R34-Pad1)
- U6 pad 2: +3V3 -> Net-(C16-Pad1)
- U6 pad 3: +10V -> Net-(U5-Pad2)
- U8 pad 3: /Front/SCL -> SCL
- U8 pad 4: /Front/SDA -> SDA
- U9 pad 14: /Front/SCL -> SCL
- U9 pad 15: /Front/SDA -> SDA

Commit message: 2021-05-13_01
Parts:
- removed H10, H11, H12, H9: MountingHole_Pad, MountingHole:MountingHole_3.2mm_M3_Pad
- removed U13: FT231XQ, Package_DFN_QFN:QFN-20-1EP_4x4mm_P0.5mm_EP2.5x2.5mm
- removed the U2 at (97.0, 33.2)
- added C31: 100nF, Capacitor_SMD:C_0603_1608Metric, F.Cu at (0.21, 58.0)
- added C32: 100uF/25V, Capacitor_THT:CP_Radial_D5.0mm_P2.00mm, F.Cu at (-20.8, 52.2)
- added C33: 10nF, Capacitor_SMD:C_0603_1608Metric, F.Cu at (-16.8, 52.2)
- added C34: X type 470pF, Capacitor_SMD:C_0603_1608Metric, F.Cu at (-2.06, 62.5)
- added D12: DB207S, Diode2:SOT4_Rectifier_Bridge, F.Cu at (60.7, 37.6)
- added D13: FR107, Diode_SMD:D_SMA, F.Cu at (45.4, 54.5)
- added D14: SS34, Diode_SMD:D_SMA, F.Cu at (54.5, 45.4)
- added H5: MountingHole_Pad, MountingHole:MountingHole_3.2mm_M3_Pad, F.Cu at (-14.8, 77.9)
- added H6: MountingHole_Pad, MountingHole:MountingHole_3.2mm_M3_Pad, F.Cu at (-14.8, 85.8)
- added H7: MountingHole_Pad, MountingHole:MountingHole_3.2mm_M3_Pad, F.Cu at (-6.85, 77.9)
- added H8: MountingHole_Pad, MountingHole:MountingHole_3.2mm_M3_Pad, F.Cu at (-6.85, 85.8)
- added HS3: Heatsink, Mechanisch:Heatsink_TO220, F.Cu at (38.2, 42.9)
- added J9: Conn_01x02, Connector2:JST_XH_B3B-XH-AM_1x03_P2.50mm_Vertical, F.Cu at (49.2, 62.6)
- added Q4: IRF840, Package_TO_SOT_THT:TO-220-3_Vertical, F.Cu at (50.5, 33.3)
- added Q5: IRF840, Package_TO_SOT_THT:TO-220-3_Vertical, F.Cu at (67.0, 39.5)
- added R42: 10k, Resistor_SMD:R_0603_1608Metric, F.Cu at (60.5, 44.4)
- added R43: 270R, Resistor_SMD:R_0603_1608Metric, F.Cu at (54.4, 53.9)
- added R44: 270R, Resistor_SMD:R_0603_1608Metric, F.Cu at (58.2, 48.9)
- added R45: 270R, Resistor_SMD:R_0603_1608Metric, F.Cu at (61.3, 41.5)
- added R46: 270R, Resistor_SMD:R_0603_1608Metric, F.Cu at (-19.8, 60.6)
- added R47: 10R, Resistor_SMD:R_2512_6332Metric, F.Cu at (0.66, 47.7)
- added R48: 300R, Resistor_SMD:R_1210_3225Metric, F.Cu at (-6.87, 62.6)
- added R49: 8k6, Resistor_SMD:R_1210_3225Metric, F.Cu at (16.4, 43.3)
- added R50: 18R, Resistor_SMD:R_1206_3216Metric, F.Cu at (6.48, 61.3)
- added R51: 150, Resistor_SMD:R_0603_1608Metric, F.Cu at (16.4, 51.2)
- added R52: 1K, Resistor_SMD:R_0603_1608Metric, F.Cu at (-13.4, 51.9)
- added R53: 22k, Resistor_SMD:R_0402_1005Metric, F.Cu at (23.6, 45.4)
- added R54: 6K8, Resistor_SMD:R_0603_1608Metric, F.Cu at (50.4, 54.2)
- added TH3: 10k_NTC, Thermistor:THERM_NXRT15XH103FA1B040, F.Cu at (53.3, 49.4)
- added U3: LM358, Package_SO:SOIC-8_3.9x4.9mm_P1.27mm, F.Cu at (46.2, 49.7)
- C1: value Y type 2N2/250VAC -> 47pF; footprint Condensator:JN_102M -> Capacitor_SMD:C_0603_1608Metric
- C10: value 10n -> 100n; footprint Capacitor_SMD:C_0402_1005Metric -> Capacitor_SMD:C_0603_1608Metric
- C11: value 6,8uF/400V -> 100n; footprint Capacitor_THT:CP_Radial_D8.0mm_P3.50mm -> Capacitor_SMD:C_0603_1608Metric
- C12: value 1nF/300V -> 100n; footprint Condensator:JN_102M -> Capacitor_SMD:C_0603_1608Metric
- C13: value 100nF/50V -> 100n
- C14: value 1000uF/25V -> 100n; footprint Capacitor_THT:CP_Radial_D10.0mm_P5.00mm -> Capacitor_SMD:C_0603_1608Metric
- C15: value 470pF/50V -> 100n
- C16: value 100nF -> Y type 2N2/250VAC; footprint Capacitor_SMD:C_0603_1608Metric -> Condensator:JN_102M
- C17: value 100uF/25V -> Y type 2N2/250VAC; footprint Capacitor_THT:CP_Radial_D5.0mm_P2.00mm -> Condensator:JN_102M
- C2: value 47pF -> 10nF; footprint Capacitor_SMD:C_0603_1608Metric -> Capacitor_SMD:C_0402_1005Metric
- C20: value 100n -> X2 100nF/275V; footprint Capacitor_SMD:C_0603_1608Metric -> Condensator:CBB22104J400V
- C21: value 100n -> 100nF
- C22: value 100n -> 4,7uF; footprint Capacitor_SMD:C_0603_1608Metric -> Capacitor_SMD:C_Elec_4x5.4
- C23: value 10nF -> 4,7uF/400V; footprint Capacitor_SMD:C_0603_1608Metric -> Capacitor_THT:CP_Radial_D8.0mm_P3.50mm
- C24: value X type 470pF -> 100n
- C26: value 100n -> 6,8uF/400V; footprint Capacitor_SMD:C_0603_1608Metric -> Capacitor_THT:CP_Radial_D8.0mm_P3.50mm
- C27: value 100n -> 1nF/300V; footprint Capacitor_SMD:C_0603_1608Metric -> Condensator:JN_102M
- C28: value 100n -> 100nF/50V
- C29: value 100nF -> 1000uF/25V; footprint Capacitor_SMD:C_0603_1608Metric -> Capacitor_THT:CP_Radial_D10.0mm_P5.00mm
- C3: value 10nF -> 47pF; footprint Capacitor_SMD:C_0402_1005Metric -> Capacitor_SMD:C_0603_1608Metric
- C30: value 4,7uF -> 470pF/50V; footprint Capacitor_SMD:C_Elec_4x5.4 -> Capacitor_SMD:C_0603_1608Metric
- C4: value Y type 2N2/250VAC -> 100nF; footprint Condensator:JN_102M -> Capacitor_SMD:C_0603_1608Metric
- C5: value 47pF -> 100uF; footprint Capacitor_SMD:C_0603_1608Metric -> Capacitor_THT:CP_Radial_D6.3mm_P2.50mm
- C6: value 100nF -> 470pF; footprint Capacitor_SMD:C_0603_1608Metric -> Capacitor_SMD:C_0402_1005Metric
- C7: value X2 100nF/275V -> 100n; footprint Condensator:CBB22104J400V -> Capacitor_SMD:C_0603_1608Metric
- C8: value 470uF/16V -> 100n; footprint Capacitor_THT:CP_Radial_D8.0mm_P3.80mm -> Capacitor_SMD:C_0603_1608Metric
- C9: value 4,7uF/400V -> 100n; footprint Capacitor_THT:CP_Radial_D8.0mm_P3.50mm -> Capacitor_SMD:C_0603_1608Metric
- D1, D7: value LED -> 3V; footprint LED_SMD:LED_0603_1608Metric_Pad1.05x0.95mm_HandSolder -> Diode_SMD:D_SMA
- D10: value SS34 -> LED; footprint Diode_SMD:D_SMA -> LED_SMD:LED_0603_1608Metric_Pad1.05x0.95mm_HandSolder
- D11, D2: footprint LED_SMD:LED_0603_1608Metric -> LED_SMD:LED_0603_1608Metric_Pad1.05x0.95mm_HandSolder
- D3: value DB207S -> 1N4148; footprint Diode2:SOT4_Rectifier_Bridge -> Diode2:DIO_LL4148
- D4: value US1K -> LED; footprint Diode_SMD:D_SMA -> LED_SMD:LED_0603_1608Metric
- D5: footprint LED_SMD:LED_0603_1608Metric_Pad1.05x0.95mm_HandSolder -> LED_SMD:LED_0603_1608Metric
- D6: value LED -> SMA12JA; footprint LED_SMD:LED_0603_1608Metric_Pad1.05x0.95mm_HandSolder -> Diode_SMD:D_SMA
- D9: value FR107 -> LED; footprint Diode_SMD:D_SMA -> LED_SMD:LED_0603_1608Metric_Pad1.05x0.95mm_HandSolder
- J3, J7: value Conn_01x02 -> Conn_01x03; footprint Connector2:JST_XH_B2B-XH-AM_1x02_P2.50mm_Vertical -> Connector2:JST_XH_B3B-XH-AM_1x03_P2.50mm_Vertical
- J4, J6: value Conn_01x03 -> Conn_01x02; footprint Connector2:JST_XH_B3B-XH-AM_1x03_P2.50mm_Vertical -> Connector2:JST_XH_B2B-XH-AM_1x02_P2.50mm_Vertical
- J5: value Conn_01x02 -> Conn_01x09_Male; footprint Connector2:JST_XH_B2B-XH-AM_1x02_P2.50mm_Vertical -> Connector_PinHeader_2.54mm:PinHeader_1x09_P2.54mm_Vertical
- J8: footprint Connector2:JST_XH_B3B-XH-AM_1x03_P2.50mm_Vertical -> Connector2:JST_XH_B2B-XH-AM_1x02_P2.50mm_Vertical
- Q1: value 4809NG -> Si2306; footprint Package_TO_SOT_THT:TO-220-3_Vertical -> Package_TO_SOT_SMD:SOT-23
- Q2: value IRF840 -> 4809NG; footprint Package_TO_SOT_THT:TO-220-3_Vertical -> Package-SOT:369AA
- Q3: value P3057G -> IRF840; footprint Package_TO_SOT_SMD:SOT-89-3 -> Package_TO_SOT_THT:TO-220-3_Vertical
- R1: value 5k6 -> 330K
- R10: value 4K7 -> 100K
- R11: value 6K8 -> 100K
- R12: value 10K -> 1K6
- R13: value 150R -> 1K6
- R14: value 100K -> 10K
- R15: value 300R -> 1K8; footprint Resistor_SMD:R_1210_3225Metric -> Resistor_SMD:R_0603_1608Metric
- R16: value 470R -> 100K
- R17: value 8k6 -> 56K; footprint Resistor_SMD:R_1210_3225Metric -> Resistor_SMD:R_0603_1608Metric
- R18: value 0R002 -> 100K; footprint Resistor_SMD:R_1206_3216Metric -> Resistor_SMD:R_0603_1608Metric
- R19: value 100k -> 33K
- R20: value 10R -> 100K
- R21: value 10R -> 10K
- R22: value 470R -> 0R
- R23: value 100k -> 100K
- R24: value 10k -> ??
- R25: value 10k -> 100K
- R26: value 10k -> 470R
- R27: value 10k -> 100k
- R28, R31: value 270R -> 0R002; footprint Resistor_SMD:R_0603_1608Metric -> Resistor_SMD:R_1206_3216Metric
- R29: value 270R -> 470R
- R30: value 270R -> 100k
- R32: value 10k -> 0R002; footprint Resistor_SMD:R_0603_1608Metric -> Resistor_SMD:R_1206_3216Metric
- R33: value 18R -> 10R; footprint Resistor_SMD:R_1206_3216Metric -> Resistor_SMD:R_0603_1608Metric
- R34: value 150 -> 10R
- R35: value 1K -> 470R
- R36: value 22k -> 100k; footprint Resistor_SMD:R_0402_1005Metric -> Resistor_SMD:R_0603_1608Metric
- R37: value 6K8 -> 0R002; footprint Resistor_SMD:R_0603_1608Metric -> Resistor_SMD:R_1206_3216Metric
- R38, R39: value 27R -> 10k
- R4: value 2K2 -> 27R
- R40, R41: value 1K6 -> 10k
- R5: value 0R002 -> 27R; footprint Resistor_SMD:R_1206_3216Metric -> Resistor_SMD:R_0603_1608Metric
- R6: value 0R002 -> 1K; footprint Resistor_SMD:R_1206_3216Metric -> Resistor_SMD:R_0603_1608Metric
- R7: value 10R -> 56K; footprint Resistor_SMD:R_2512_6332Metric -> Resistor_SMD:R_0603_1608Metric
- R8: value 10K -> 4K7
- RV1: value 10D431K -> 10K; footprint Varistor2:RV_Disc_D10mm_W2mm_P8mm -> Potentiometer_THT:Potentiometer_Bourns_3266Y_Vertical
- RV2: value 10K -> 10D431K; footprint Potentiometer_THT:Potentiometer_Bourns_3296W_Vertical -> Varistor2:RV_Disc_D10mm_W2mm_P8mm
- TH1, TH2: footprint Capacitor_THT:C_Disc_D3.8mm_W2.6mm_P2.50mm -> Thermistor:THERM_NXRT15XH103FA1B040
- U10: value MCP4725A0 -> PC817; footprint Package_TO_SOT_SMD:SOT-23-6 -> Package_SO:SSO-4_6.7x5.1mm_P2.54mm_Clearance8mm
- U2: renamed from U3; value LM358 -> FT231XQ; footprint Package_SO:SOIC-8_3.9x4.9mm_P1.27mm -> Package_DFN_QFN:QFN-20-1EP_4x4mm_P0.5mm_EP2.5x2.5mm
- U5: value LNK364D -> LM358; footprint Package_SO:PowerIntegrations_SO-8C -> Package_SO:SOIC-8_3.9x4.9mm_P1.27mm
- U6: value PC817 -> (none); footprint Package_SO:SSO-4_6.7x5.1mm_P2.54mm_Clearance8mm -> Package_SO:SOIC-8_3.9x4.9mm_P1.27mm
- U7: value LM358 -> PCF8574; footprint Package_SO:SOIC-8_3.9x4.9mm_P1.27mm -> Package_SO:SOIC-16W_7.5x10.3mm_P1.27mm
- U9: value PCF8574 -> LNK364D; footprint Package_SO:SOIC-16W_7.5x10.3mm_P1.27mm -> Package_SO:PowerIntegrations_SO-8C
- moved R1 97.3 mm to (58.2, 51.4)
- moved D4 82.4 mm to (-16.5, 45.8)
- moved C25 75.6 mm to (-8.68, 55.7)
- moved C12 73.7 mm to (-30.5, 55.9)
- moved C10 71.6 mm to (6.48, 58.8)
- moved C4 71.1 mm to (69.7, 33.3)
- moved C17 66.1 mm to (7.03, 42.4)
- moved C7 65.8 mm to (66.1, 43.0)
- moved D3 64.8 mm to (62.8, 31.6)
- moved R13 63.3 mm to (62.2, 46.9)
- moved C26 62.4 mm to (-1.59, 31.7)
- moved C15 61.2 mm to (13.5, 48.7)
- moved D10 61.0 mm to (1.87, 52.4)
- moved C28 60.5 mm to (-4.46, 39.8)
- moved U4 58.0 mm to (17.9, 76.2)
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Connections:
- C1 pad 1: Earth -> Net-(C1-Pad1)
- C1 pad 2: Net-(C1-Pad2) -> GND
- C10 pad 1: GNDA -> GND
- C11 pad 1: Net-(C11-Pad1) -> GNDA
- C11 pad 2: Net-(C11-Pad2) -> VDC
- C12 pad 1: Net-(C11-Pad1) -> GNDA
- C12 pad 2: Net-(C12-Pad2) -> VDC
- C13 pad 1: Net-(C13-Pad1) -> GND
- C13 pad 2: Net-(C11-Pad2) -> +3V3
- C14 pad 1: Net-(C14-Pad1) -> GND
- C14 pad 2: GND -> +3V3
- C15 pad 1: Net-(C14-Pad1) -> GND
- C15 pad 2: Net-(C15-Pad2) -> +3V3
- C16 pad 1: Net-(C16-Pad1) -> Earth
- C17 pad 1: +12V -> NEUTRAL
- C17 pad 2: GND -> Earth
- C18 pad 2: Net-(C18-Pad2) -> +3V3
- C19 pad 1: Net-(C19-Pad1) -> GND
- C19 pad 2: Net-(C19-Pad2) -> +3V3
- C20 pad 1: GND -> Net-(C20-Pad1)
- C20 pad 2: Net-(C20-Pad2) -> NEUTRAL
- C21 pad 1: GNDA -> VCC
- C21 pad 2: VDC -> GND
- C22 pad 1: GNDA -> VCC
- C22 pad 2: VDC -> GND
- C23 pad 1: +12V -> Net-(C23-Pad1)
- C23 pad 2: GND -> Net-(C23-Pad2)
- C24 pad 1: Earth -> GND
- C24 pad 2: GND -> +12V
- C25 pad 2: +3V3 -> +12V
- C26 pad 1: GND -> Net-(C26-Pad1)
- C26 pad 2: +3V3 -> Net-(C26-Pad2)
- C27 pad 1: GND -> Net-(C26-Pad1)
- C27 pad 2: +3V3 -> Net-(C27-Pad2)
- C28 pad 1: GND -> Net-(C28-Pad1)
- C28 pad 2: +3V3 -> Net-(C26-Pad2)
- C29 pad 1: VCC -> Net-(C29-Pad1)
- C30 pad 1: VCC -> Net-(C29-Pad1)
- C30 pad 2: GND -> Net-(C30-Pad2)
- C4 pad 1: NEUTRAL -> Net-(C4-Pad1)
- C4 pad 2: Earth -> GND
- C5 pad 1: Net-(C5-Pad1) -> +3V3
- C5 pad 2: GND -> Net-(C5-Pad2)
- C6 pad 2: GND -> Net-(C6-Pad2)
- C7 pad 1: Net-(C7-Pad1) -> GND
- C7 pad 2: NEUTRAL -> Net-(C7-Pad2)
- C8 pad 1: Net-(C8-Pad1) -> GND
- C8 pad 2: GNDA -> Net-(C8-Pad2)
- D1 pad 1: Net-(D1-Pad1) -> ADC
- D1 pad 2: Net-(D1-Pad2) -> GND
- D10 pad 1: Net-(C14-Pad1) -> Net-(D10-Pad1)
- D3 pad 1: NEUTRAL -> Net-(D3-Pad1)
- D3 pad 2: Net-(C7-Pad1) -> GND
- D4 pad 1: Net-(C8-Pad1) -> Net-(D4-Pad1)
- D4 pad 2: GNDA -> Net-(D4-Pad2)
- D6 pad 1: Net-(D6-Pad1) -> +12V
- D7 pad 1: Net-(D7-Pad1) -> FAN_TACH
- F1 pad 1: Net-(C1-Pad2) -> Net-(C16-Pad2)
- FB1 pad 2: Net-(C3-Pad1) -> Net-(C2-Pad1)
- J1 pad A4: Net-(C3-Pad1) -> Net-(C2-Pad1)
- J1 pad A6: Net-(C5-Pad1) -> Net-(C3-Pad1)
- J1 pad A7: Net-(C2-Pad1) -> Net-(C1-Pad1)
- J1 pad A9: Net-(C3-Pad1) -> Net-(C2-Pad1)
- J1 pad B4: Net-(C3-Pad1) -> Net-(C2-Pad1)
- J1 pad B6: Net-(C5-Pad1) -> Net-(C3-Pad1)
- J1 pad B7: Net-(C2-Pad1) -> Net-(C1-Pad1)
- J1 pad B9: Net-(C3-Pad1) -> Net-(C2-Pad1)
- J2 pad 1: Net-(C8-Pad1) -> Net-(D7-Pad2)
- J2 pad 2: GNDA -> +12V
- J3 pad 1: LOAD -> SCL
- J3 pad 2: GND -> Net-(J3-Pad2)
- J4 pad 1: SCL -> VDC
- J4 pad 2: ~INT -> GNDA
- J5 pad 1: +3V3 -> Net-(J5-Pad1)
- J5 pad 2: GND -> Net-(J5-Pad2)
- J6 pad 1: SCL -> LOAD
- J6 pad 2: Net-(J6-Pad2) -> GND
- J7 pad 1: VDC -> SCL
- J7 pad 2: GNDA -> ~INT
- J8 pad 1: LINE -> +3V3
- J8 pad 2: Earth -> GND
- L1 pad 1: Net-(C9-Pad1) -> Net-(C23-Pad1)
- L1 pad 2: Net-(C9-Pad2) -> Net-(C23-Pad2)
- L1 pad 3: Net-(C11-Pad2) -> Net-(C26-Pad2)
- L1 pad 4: Net-(C11-Pad1) -> Net-(C26-Pad1)
- L2 pad 1: Net-(C14-Pad1) -> Net-(C29-Pad1)
- Q1 pad 1: Net-(C18-Pad2) -> Net-(C5-Pad2)
- Q1 pad 2: LOAD -> GND
- Q1 pad 3: Net-(Q1-Pad3) -> THERM
- Q2 pad 1: Net-(C20-Pad2) -> Net-(Q2-Pad1)
- Q2 pad 2: LOAD -> Net-(D6-Pad2)
- Q2 pad 3: Net-(Q2-Pad3) -> Net-(D7-Pad2)
- Q3 pad 1: Net-(Q3-Pad1) -> Net-(C7-Pad2)
- Q3 pad 2: +12V -> LOAD
- Q3 pad 3: Net-(C8-Pad1) -> Net-(Q3-Pad3)
- R1 pad 1: THERM -> LOAD
- R1 pad 2: GND -> ADC
- R10 pad 1: SDA -> Net-(R10-Pad1)
- R10 pad 2: +3V3 -> +5V
- R11 pad 1: GNDA -> Net-(C6-Pad1)
- R11 pad 2: Net-(R11-Pad2) -> Net-(R10-Pad1)
- R12 pad 1: Net-(C8-Pad1) -> Net-(D4-Pad2)
- R12 pad 2: Net-(R11-Pad2) -> VCC
- R13 pad 1: Net-(Q3-Pad1) -> Net-(D5-Pad2)
- R13 pad 2: Net-(C10-Pad2) -> VCC
- R14 pad 1: Net-(C8-Pad1) -> Net-(R10-Pad1)
- R14 pad 2: Net-(Q3-Pad1) -> Net-(R14-Pad2)
- R15 pad 1: Net-(C12-Pad2) -> Net-(C6-Pad2)
- R15 pad 2: Net-(D9-Pad1) -> Net-(R14-Pad2)
- R16 pad 1: Net-(R16-Pad1) -> GND
- R16 pad 2: Net-(C18-Pad2) -> Net-(R16-Pad2)
- R17 pad 1: Net-(C11-Pad1) -> Net-(R17-Pad1)
- R17 pad 2: Net-(C12-Pad2) -> Net-(R16-Pad2)
- R18 pad 1: GND -> Net-(R18-Pad1)
- R18 pad 2: SHUNT -> +12V
- R19 pad 1: Net-(C18-Pad2) -> GND
- R19 pad 2: Net-(Q1-Pad3) -> Net-(R18-Pad1)
- R2 pad 1: +3V3 -> ADC
- R2 pad 2: RTS -> GND
- R20 pad 1: Net-(C19-Pad1) -> Net-(D7-Pad2)
- R20 pad 2: SHUNT -> Net-(Q2-Pad1)
- R21 pad 1: Net-(C19-Pad2) -> Net-(R21-Pad1)
- R21 pad 2: GND -> Net-(R17-Pad1)
- R22 pad 1: Net-(R16-Pad1) -> Net-(R18-Pad1)
- R22 pad 2: Net-(C20-Pad2) -> Net-(R21-Pad1)
- R23 pad 1: Net-(C20-Pad2) -> GND
- R23 pad 2: Net-(Q2-Pad3) -> Net-(R23-Pad2)
- R24 pad 1: VDC -> Net-(D6-Pad2)
- R24 pad 2: Net-(R24-Pad2) -> +12V
- R25 pad 1: VDC -> Net-(R25-Pad1)
- R25 pad 2: Net-(R25-Pad2) -> Net-(R23-Pad2)
- R26 pad 1: VDC -> Net-(R25-Pad1)
- R26 pad 2: Net-(R26-Pad2) -> Net-(C7-Pad2)
- R27 pad 1: VDC -> Net-(C7-Pad2)
- R27 pad 2: Net-(R27-Pad2) -> Net-(Q3-Pad3)
- R28 pad 1: Net-(D5-Pad1) -> SHUNT
- R28 pad 2: GNDA -> Net-(Q3-Pad3)
- R29 pad 1: Net-(D6-Pad1) -> Net-(R25-Pad1)
- R29 pad 2: GNDA -> Net-(C8-Pad2)
- R3 pad 1: Net-(D1-Pad1) -> Net-(D2-Pad1)
- R30 pad 1: Net-(D7-Pad1) -> Net-(C8-Pad2)
- R30 pad 2: GNDA -> Net-(Q4-Pad3)
- R31 pad 1: Net-(D8-Pad1) -> GND
- R31 pad 2: GNDA -> SHUNT
- R32 pad 1: VDC -> SHUNT
- R32 pad 2: Net-(J6-Pad2) -> Net-(Q4-Pad3)
- R33 pad 1: Net-(C15-Pad2) -> Net-(C9-Pad1)
- R33 pad 2: Net-(D10-Pad2) -> SHUNT
- R34 pad 1: Net-(R34-Pad1) -> Net-(C9-Pad2)
- R34 pad 2: Net-(C14-Pad1) -> GND
- R35 pad 1: Net-(R34-Pad1) -> Net-(R25-Pad1)
- R35 pad 2: Net-(C16-Pad1) -> Net-(C10-Pad2)
- R36 pad 1: +12V -> Net-(C10-Pad2)
- R36 pad 2: Net-(C16-Pad2) -> Net-(Q5-Pad3)
- R37 pad 1: Net-(C16-Pad2) -> SHUNT
- R37 pad 2: GND -> Net-(Q5-Pad3)
- R38 pad 1: Net-(R38-Pad1) -> VDC
- R38 pad 2: Net-(C2-Pad1) -> Net-(J3-Pad2)
- R39 pad 1: Net-(R39-Pad1) -> VDC
- R39 pad 2: Net-(C5-Pad1) -> Net-(R39-Pad2)
- R4 pad 2: GND -> Net-(C1-Pad1)
- R40 pad 1: Net-(D11-Pad2) -> VDC
- R40 pad 2: VCC -> Net-(R40-Pad2)
- R41 pad 1: Net-(D2-Pad2) -> VDC
- R41 pad 2: VCC -> Net-(R41-Pad2)
- R5 pad 1: SHUNT -> Net-(R5-Pad1)
- R5 pad 2: Net-(Q1-Pad3) -> Net-(C3-Pad1)
- R6 pad 1: SHUNT -> Net-(D3-Pad1)
- R6 pad 2: Net-(Q2-Pad3) -> Net-(C5-Pad2)
- R7 pad 1: Net-(C7-Pad1) -> GND
- R7 pad 2: Net-(C1-Pad2) -> Net-(C5-Pad2)
- R8 pad 1: GNDA -> SCL
- R8 pad 2: Net-(R8-Pad2) -> +3V3
- R9 pad 1: SCL -> SDA
- RV1 pad 1: Net-(C1-Pad2) -> Net-(RV1-Pad1)
- RV1 pad 2: NEUTRAL -> +5V
- RV2 pad 1: Net-(R16-Pad1) -> Net-(C16-Pad2)
- RV2 pad 2: Net-(R4-Pad1) -> NEUTRAL
- SW1 pad 1: Net-(R24-Pad2) -> Net-(R39-Pad2)
- SW1 pad 2: Net-(R24-Pad2) -> Net-(R39-Pad2)
- SW2 pad 1: Net-(R25-Pad2) -> Net-(R40-Pad2)
- SW2 pad 2: Net-(R25-Pad2) -> Net-(R40-Pad2)
- SW3 pad 1: Net-(R26-Pad2) -> Net-(R41-Pad2)
- SW3 pad 2: Net-(R26-Pad2) -> Net-(R41-Pad2)
- SW4 pad 1: Net-(R27-Pad2) -> Net-(R42-Pad2)
- SW4 pad 2: Net-(R27-Pad2) -> Net-(R42-Pad2)
- T1 pad 1: Net-(C11-Pad1) -> Net-(C26-Pad1)
- T1 pad 2: Net-(D9-Pad2) -> Net-(D13-Pad2)
- T1 pad 4: Net-(D10-Pad2) -> Net-(D14-Pad2)
- TH1 pad 1: +3V3 -> THERM
- TH1 pad 2: THERM -> GND
- TH2 pad 1: +3V3 -> THERM
- TH2 pad 2: THERM -> GND
- U1 pad 2: THERM -> ADC
- U1 pad 5: Net-(U1-Pad5) -> FAN_TACH
- U1 pad 7: Net-(D1-Pad2) -> Net-(D2-Pad2)
- U10 pad 1: Net-(U10-Pad1) -> Net-(R51-Pad1)
- U10 pad 2: GND -> Net-(C31-Pad1)
- U10 pad 3: +3V3 -> Net-(U10-Pad3)
- U10 pad 4: SDA -> Net-(C28-Pad1)
- U11 pad 1: Net-(C16-Pad1) -> Net-(C31-Pad1)
- U11 pad 2: Net-(C16-Pad2) -> Net-(C31-Pad2)
- U2 pad 1: Net-(R16-Pad1) -> TX
- U2 pad 2: Net-(R4-Pad1) -> Net-(U2-Pad2)
- U2 pad 3: Net-(U10-Pad1) -> GND
- U2 pad 4: (no net) -> Net-(U2-Pad4)
- U2 pad 5: Net-(R8-Pad2) -> Net-(U2-Pad5)
- U2 pad 6: Net-(R11-Pad2) -> Net-(U2-Pad6)
- U2 pad 7: Net-(C10-Pad2) -> Net-(D5-Pad1)
- U2 pad 8: (no net) -> Net-(R5-Pad1)
- U4 pad 1: Net-(R8-Pad2) -> Net-(U4-Pad1)
- U4 pad 2: GNDA -> GND
- U4 pad 6: +3V3 -> GND
- U5 pad 1: Net-(C13-Pad1) -> Net-(R17-Pad1)
- U5 pad 2: Net-(U5-Pad2) -> Net-(R16-Pad2)
- U5 pad 4: Net-(D9-Pad2) -> GND
- U5 pad 5: Net-(C11-Pad2) -> Net-(R21-Pad1)
- U5 pad 6: Net-(C11-Pad2) -> Net-(R23-Pad2)
- U5 pad 7: Net-(C11-Pad2) -> Net-(R25-Pad1)
- U5 pad 8: Net-(C11-Pad2) -> +5V
- U6 pad 1: Net-(R34-Pad1) -> GND
- U6 pad 2: Net-(C16-Pad1) -> GND
- U6 pad 3: Net-(U5-Pad2) -> SDA
- U6 pad 4: Net-(C13-Pad1) -> SCL
- U7 pad 1: GND -> GNDA
- U7 pad 2: GND -> GNDA
- U7 pad 3: SDA -> GNDA
- U7 pad 4: SCL -> Net-(R39-Pad2)
- U7 pad 5: +3V3 -> Net-(R40-Pad2)
- U7 pad 6: GND -> Net-(R41-Pad2)
- U7 pad 7: Net-(C19-Pad2) -> Net-(R42-Pad2)
- U7 pad 8: Net-(C19-Pad1) -> GNDA
- U9 pad 1: GNDA -> Net-(C28-Pad1)
- U9 pad 2: GNDA -> Net-(U10-Pad3)
- U9 pad 4: Net-(R24-Pad2) -> Net-(D13-Pad2)
- U9 pad 5: Net-(R25-Pad2) -> Net-(C26-Pad2)
- U9 pad 6: Net-(R26-Pad2) -> Net-(C26-Pad2)
- U9 pad 7: Net-(R27-Pad2) -> Net-(C26-Pad2)
- U9 pad 8: GNDA -> Net-(C26-Pad2)

Commit message: 2021-05-14_02
Parts:
- removed D10, D11, D8, D9: LED, LED_SMD:LED_0603_1608Metric_Pad1.05x0.95mm_HandSolder
- removed SW1, SW2, SW3, SW4: Switch_6x6_SMT, Switches:SW_SPST_6x6x20mm_SMD
- added J10: Conn_01x02, Connector2:JST_XH_B2B-XH-AM_1x02_P2.50mm_Vertical, F.Cu at (136.8, 46.3)
- added Q6: Si2306, Package_TO_SOT_SMD:SOT-23, F.Cu at (145.1, 48.5)
- added R55: 10k, Resistor_SMD:R_0603_1608Metric, B.Cu at (125.0, 133.9)
- added R56: 10k, Resistor_SMD:R_0603_1608Metric, B.Cu at (127.9, 133.9)
- D1, D7: value 3V -> BZT52C-3V6; footprint Diode_SMD:D_SMA -> Diode_SMD:D_SOD-123
- J2: footprint Connector2:JST_XH_B2B-XH-AM_1x02_P2.50mm_Vertical -> Connector_JST:JST_XH_B4B-XH-A_1x04_P2.50mm_Vertical
- J3, J4, J5, R38, R39, R40, R41, R42, U7: moved to B.Cu
- J7: moved to F.Cu
- R24: value ?? -> 1K
- R43: value 270R -> 10K
- R44: value 270R -> 4K7
- R45, R46: value 270R -> 10k; moved to B.Cu
- moved H8 166.6 mm to (147.0, 149.7)
- moved J8 166.3 mm to (210.9, 96.5)
- moved H7 162.2 mm to (147.7, 127.1)
- moved R46 159.7 mm to (122.1, 133.9), turned to 270 degrees
- moved C11 129.1 mm to (61.2, 142.9)
- moved J3 128.9 mm to (136.9, 135.7), turned to 90 degrees
- moved J4 125.3 mm to (136.9, 146.3), turned to 90 degrees
- moved C12 115.0 mm to (59.9, 127.0)
- moved J5 110.7 mm to (107.8, 147.8), turned to 270 degrees
- moved R45 109.3 mm to (119.7, 133.9), turned to 270 degrees
- moved H6 108.0 mm to (72.1, 149.9)
- moved H5 100.0 mm to (72.0, 127.5)
- moved D7 99.8 mm to (145.7, 44.6)
- moved R40 99.7 mm to (98.7, 133.9), turned to 270 degrees
- moved R42 99.7 mm to (104.4, 133.9), turned to 270 degrees
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Connections:
- D7 pad 1: FAN_TACH -> Net-(D7-Pad1)
- D7 pad 2: Net-(D7-Pad2) -> GND
- J1 pad A5: Net-(J1-PadA5) -> (no net)
- J1 pad A8: Net-(J1-PadA8) -> (no net)
- J1 pad B5: Net-(J1-PadB5) -> (no net)
- J1 pad B8: Net-(J1-PadB8) -> (no net)
- J2 pad 1: Net-(D7-Pad2) -> GND
- J3 pad 1: SCL -> /Front/SCL
- J3 pad 3: SDA -> /Front/SDA
- J5 pad 9: Net-(J5-Pad9) -> (no net)
- Q2 pad 3: Net-(D7-Pad2) -> GND
- R20 pad 1: Net-(D7-Pad2) -> GND
- R39 pad 2: Net-(R39-Pad2) -> Net-(J5-Pad1)
- R40 pad 2: Net-(R40-Pad2) -> Net-(J5-Pad2)
- R41 pad 2: Net-(R41-Pad2) -> Net-(J5-Pad3)
- R42 pad 2: Net-(R42-Pad2) -> Net-(J5-Pad4)
- R43 pad 1: Net-(D8-Pad1) -> Net-(D7-Pad1)
- R43 pad 2: GNDA -> +3V3
- R44 pad 1: Net-(D9-Pad1) -> Net-(D7-Pad1)
- R44 pad 2: GNDA -> FAN_TACH
- R45 pad 1: Net-(D10-Pad1) -> VDC
- R45 pad 2: GNDA -> Net-(J5-Pad8)
- R46 pad 1: Net-(D11-Pad1) -> VDC
- R46 pad 2: GNDA -> Net-(J5-Pad7)
- RV1 pad 1: Net-(RV1-Pad1) -> (no net)
- U1 pad 10: Net-(U1-Pad10) -> (no net)
- U1 pad 11: Net-(U1-Pad11) -> (no net)
- U1 pad 17: Net-(U1-Pad17) -> (no net)
- U1 pad 18: Net-(U1-Pad18) -> (no net)
- U1 pad 19: Net-(U1-Pad19) -> (no net)
- U1 pad 20: Net-(U1-Pad20) -> (no net)
- U1 pad 21: Net-(U1-Pad21) -> (no net)
- U1 pad 22: Net-(U1-Pad22) -> (no net)
- U1 pad 6: Net-(U1-Pad6) -> FAN_OVERRIDE
- U2 pad 15: Net-(U2-Pad15) -> (no net)
- U2 pad 16: Net-(U2-Pad16) -> (no net)
- U2 pad 2: Net-(U2-Pad2) -> (no net)
- U2 pad 4: Net-(U2-Pad4) -> (no net)
- U2 pad 5: Net-(U2-Pad5) -> (no net)
- U2 pad 6: Net-(U2-Pad6) -> (no net)
- U7 pad 10: Net-(D10-Pad2) -> Net-(J5-Pad7)
- U7 pad 11: Net-(D9-Pad2) -> Net-(J5-Pad6)
- U7 pad 12: Net-(D8-Pad2) -> Net-(J5-Pad5)
- U7 pad 14: SCL -> /Front/SCL
- U7 pad 15: SDA -> /Front/SDA
- U7 pad 4: Net-(R39-Pad2) -> Net-(J5-Pad1)
- U7 pad 5: Net-(R40-Pad2) -> Net-(J5-Pad2)
- U7 pad 6: Net-(R41-Pad2) -> Net-(J5-Pad3)
- U7 pad 7: Net-(R42-Pad2) -> Net-(J5-Pad4)
- U7 pad 9: Net-(D11-Pad2) -> Net-(J5-Pad8)
- U8 pad 3: SCL -> /Front/SCL
- U8 pad 4: SDA -> /Front/SDA
Routing:
- net VDC: track 0.00 -> 19.7 mm
- net Net-(J3-Pad2): track 0.00 -> 17.5 mm
- net Net-(J5-Pad1): track 0.00 -> 14.9 mm
- net Net-(J5-Pad5): track 0.00 -> 13.5 mm
- net Net-(J5-Pad2): track 0.00 -> 10.8 mm
- net Net-(J5-Pad6): track 0.00 -> 9.39 mm
- net Net-(J5-Pad3): track 0.00 -> 6.61 mm
- net Net-(J5-Pad7): track 0.00 -> 2.95 mm
- net Net-(J5-Pad4): track 0.00 -> 2.95 mm
Other:
- board text added: "ENA"
- board text added: "GND"
- board text added: "SCL"
- board text added: "SDA"
- board text added: "VDC"

Commit message: 2021-05-15_01
Parts:
- C11, C12: moved to B.Cu
- J6: moved to F.Cu
- moved J8 92.3 mm to (120.1, 113.0)
- moved RV2 91.8 mm to (171.5, 51.0)
- moved J9 90.4 mm to (139.6, 64.5), turned to 180 degrees
- moved U1 88.9 mm to (-13.7, 96.2)
- moved Q3 86.4 mm to (95.6, 109.7), turned to 90 degrees
- moved Q4 74.1 mm to (95.6, 92.1), turned to 90 degrees
- moved TH2 73.7 mm to (89.3, 89.7), turned to 270 degrees
- moved H4 69.4 mm to (72.1, 62.0)
- moved J7 66.1 mm to (135.0, 113.0)
- moved J6 65.0 mm to (103.2, 112.8)
- moved HS3 58.9 mm to (89.3, 72.2), turned to 90 degrees
- moved H3 58.3 mm to (72.1, 116.9)
- moved J2 57.5 mm to (109.4, 64.5), turned to 180 degrees
- moved Q5 45.4 mm to (95.6, 74.7), turned to 90 degrees
- moved TH3 42.6 mm to (89.3, 72.2), turned to 270 degrees
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Routing:
- net /Front/SDA: track 0.00 -> 65.5 mm, vias 0 -> 1
- net /Front/SCL: track 0.00 -> 56.2 mm, vias 0 -> 1
- net Net-(J5-Pad5): track 13.5 -> 63.6 mm
- net VDC: track 19.7 -> 64.4 mm
- net Net-(J5-Pad8): track 0.07 -> 37.1 mm
- net Net-(J5-Pad7): track 2.95 -> 38.6 mm
- net Net-(J5-Pad4): track 2.95 -> 36.3 mm
- net Net-(J5-Pad6): track 9.39 -> 37.9 mm
- net Net-(J5-Pad3): track 6.61 -> 34.6 mm
- net Net-(J5-Pad2): track 10.8 -> 33.3 mm
- net Net-(J3-Pad2): track 17.5 -> 38.0 mm, vias 0 -> 1
- net Net-(J5-Pad1): track 14.9 -> 31.2 mm
- net GNDA: track 0.00 -> 3.69 mm, vias 0 -> 2
- added copper zone on B.Cu, net GNDA
- added copper zone on F.Cu, net GNDA
Other:
- outline, holes or cut-outs redrawn
- rule pad_to_mask_clearance: 0 -> 0.051
- rule trace_min: 0.1 -> 0.1016
- rule via_min_size: 0.4 -> 0.3048
- board text added: "230V"
- board text added: "3V3"
- board text added: "INT"
- board text added: "LINE"
- board text added: "LOAD"
- board text added: "NEUT"

Commit message: 2021-05-15_02
Parts:
- added C35: 100n, Capacitor_SMD:C_0603_1608Metric, F.Cu at (106.6, 108.1)
- C21, R26, R27, R32: moved to F.Cu
- moved D4 133.4 mm to (114.5, 70.4)
- moved U5 114.8 mm to (109.1, 103.6), turned to 180 degrees
- moved C13 112.8 mm to (128.7, 74.8)
- moved U4 111.1 mm to (127.2, 95.6)
- moved R27 108.9 mm to (98.1, 108.8), turned to 90 degrees
- moved C8 94.9 mm to (97.3, 96.6)
- moved C10 93.1 mm to (97.3, 79.1)
- moved R32 91.1 mm to (99.6, 87.0), turned to 180 degrees
- moved R28 84.6 mm to (99.6, 104.6), turned to 180 degrees
- moved R30 84.5 mm to (98.1, 91.2), turned to 90 degrees
- moved R25 84.2 mm to (104.2, 103.5), turned to 90 degrees
- moved D5 82.1 mm to (114.5, 74.0), turned to 0 degrees
- moved R26 80.8 mm to (100.6, 107.1), turned to 180 degrees
- moved R29 78.1 mm to (97.3, 98.4), turned to 180 degrees
- moved C21 77.4 mm to (117.1, 75.0), turned to 270 degrees
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Connections:
- R18 pad 2: +12V -> +5V
Routing:
- net LOAD: track 0.00 -> 57.1 mm
- net Net-(R25-Pad1): track 0.00 -> 35.9 mm
- net SHUNT: track 0.00 -> 35.0 mm
- net Net-(C2-Pad1): track 0.00 -> 13.5 mm
- net Net-(R18-Pad1): track 0.00 -> 13.0 mm
- net Net-(R17-Pad1): track 0.00 -> 11.5 mm
- net (no net): track 0.00 -> 10.6 mm
- net Net-(C8-Pad2): track 0.00 -> 9.57 mm
- net Net-(C10-Pad2): track 0.00 -> 9.36 mm
- net Net-(C3-Pad1): track 0.00 -> 8.93 mm
- net Net-(C7-Pad2): track 0.00 -> 6.38 mm
- net Net-(Q3-Pad3): track 0.00 -> 5.94 mm
- net Net-(R4-Pad1): track 0.00 -> 5.93 mm
- net Net-(R16-Pad2): track 0.00 -> 5.06 mm
- net Net-(C1-Pad1): track 0.00 -> 4.74 mm
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
Commit message: 2021-05-16_01
Parts:
- R24: moved to F.Cu
- moved U1 151.1 mm to (136.7, 110.2), turned to 180 degrees
- moved RV1 138.4 mm to (116.5, 88.8), turned to 270 degrees
- moved U6 137.3 mm to (108.9, 93.0)
- moved C15 116.2 mm to (114.2, 106.8), turned to 90 degrees
- moved C24 112.0 mm to (112.0, 83.5)
- moved C9 104.6 mm to (110.3, 97.0)
- moved R6 77.9 mm to (50.9, 88.6)
- moved R7 73.9 mm to (116.2, 100.0), turned to 90 degrees
- moved U3 73.8 mm to (109.8, 87.2)
- moved R31 73.6 mm to (103.5, 92.7), turned to 270 degrees
- moved C19 73.1 mm to (56.1, 103.7)
- moved R9 73.1 mm to (52.1, 102.9)
- moved R3 72.4 mm to (58.5, 97.6)
- moved C18 72.4 mm to (53.8, 94.0)
- moved R24 67.6 mm to (103.0, 69.6)
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Routing:
- net THERM: track 0.00 -> 80.1 mm, vias 0 -> 1
- net Net-(C6-Pad2): track 0.00 -> 14.8 mm
- net Net-(R10-Pad1): track 0.00 -> 14.3 mm
- net Net-(C9-Pad2): track 0.00 -> 9.30 mm
- net Net-(C9-Pad1): track 0.00 -> 9.02 mm
- net LOAD: track 57.1 -> 48.3 mm
- net VCC: track 0.00 -> 8.38 mm
- net GND: track 0.60 -> 8.48 mm, vias 0 -> 3
- net SHUNT: track 35.0 -> 41.9 mm
- net Net-(D4-Pad1): track 0.00 -> 5.06 mm
- net Net-(D5-Pad1): track 0.00 -> 4.49 mm
- net Net-(R14-Pad2): track 0.00 -> 4.29 mm
- net Net-(R4-Pad1): track 5.93 -> 2.42 mm
- net +3V3: track 0.00 -> 3.23 mm
- net Net-(Q5-Pad3): track 3.49 -> 6.04 mm
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