File: NieuwOntwerp/Load.kicad_pcb (KiCad board)
At the start: 2 copper layers, 84 x 96 mm, 150 parts, among them J1 USB_C_Receptacle_USB2.0, J10 Conn_01x02, J2 Conn_01x02, J3 Conn_01x03, J4 Conn_01x02, J5 Conn_01x09_Male, J6 Conn_01x02, J7 Conn_01x03, J8 Conn_01x02, J9 Conn_01x02, Q1 Si2306, Q2 4809NG, Q3 IRF840, Q4 IRF840, Q5 IRF840, Q6 Si2306, T1 EE13, U1 ESP12E, U10 PC817, U11 TL431, U12 LM1117-3.3, U2 FT231XQ, U3 LM358, U4 MCP4725A0, U5 LM358, U6 , U7 PCF8574, U8 SSD1306, U9 LNK364D

Commit message: start
Parts:
- removed C14, C18, C25: 100n, Capacitor_SMD:C_0603_1608Metric
- added D10: MMSZ5225/3V, Diode_SMD:D_SOD-123, F.Cu at (26.8, -5.29)
- added D8: BZT52C-5V1, Diode_SMD:D_SOD-123, F.Cu at (60.5, 63.2)
- added D9: MMSZ5225/3V, Diode_SMD:D_SOD-123, F.Cu at (26.8, -8.64)
- added R57: 1K2, Resistor_SMD:R_0603_1608Metric, F.Cu at (57.0, 63.5)
- C16, C17: footprint Condensator:JN_102M -> Condensator:Y2_222
- C22, U9: moved to F.Cu
- C34: footprint Capacitor_SMD:C_0603_1608Metric -> Condensator:JN_102M
- C5: footprint Capacitor_THT:CP_Radial_D6.3mm_P2.50mm -> Capacitor_THT:CP_Radial_D5.0mm_P2.00mm
- F1: footprint Fuse:Fuse_1206_3216Metric -> FuseClip:fuse-clip-5x20mm
- R48: value 300R -> 330R; footprint Resistor_SMD:R_1210_3225Metric -> Resistor_THT:R_Axial_DIN0207_L6.3mm_D2.5mm_P2.54mm_Vertical
- R49: footprint Resistor_SMD:R_1210_3225Metric -> Resistor_THT:R_Axial_DIN0207_L6.3mm_D2.5mm_P2.54mm_Vertical
- T1: footprint Transformers:EE13Horizontal -> Transformers:EE16-A2
- U6: value (none) -> INA219; footprint Package_SO:SOIC-8_3.9x4.9mm_P1.27mm -> Package_TO_SOT_SMD:SOT-23-8
- moved U9 127.6 mm to (76.2, 38.8), turned to 90 degrees
- moved L1 114.6 mm to (85.3, 26.8)
- moved T1 114.0 mm to (84.1, 49.2), turned to 90 degrees
- moved R20 111.6 mm to (38.4, 19.4), turned to 180 degrees
- moved RV2 104.5 mm to (71.2, 21.8), turned to 270 degrees
- moved D7 103.7 mm to (44.3, 23.0), turned to 90 degrees
- moved U1 101.9 mm to (60.4, 42.7)
- moved J9 100.3 mm to (57.8, 6.48), turned to 270 degrees
- moved R48 99.3 mm to (89.9, 40.6), turned to 180 degrees
- moved R2 99.2 mm to (64.4, 40.7)
- moved R44 96.6 mm to (47.2, 23.1)
- moved C20 96.2 mm to (64.9, 16.0), turned to 270 degrees
- moved C35 95.5 mm to (28.4, 53.3)
- moved R13 94.8 mm to (47.2, 18.2), turned to 0 degrees
- moved R7 94.0 mm to (39.8, 45.2)
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Connections:
- D12 pad 1: NEUTRAL -> Net-(C23-Pad1)
- D12 pad 2: Net-(C20-Pad1) -> Net-(C23-Pad2)
- D12 pad 3: Net-(C23-Pad1) -> Net-(C20-Pad1)
- D12 pad 4: Net-(C23-Pad2) -> NEUTRAL
- H2 pad 1: GND -> Net-(H2-Pad1)
- J1 pad A5: (no net) -> Net-(J1-PadA5)
- J1 pad A8: (no net) -> Net-(J1-PadA8)
- J1 pad B5: (no net) -> Net-(J1-PadB5)
- J1 pad B8: (no net) -> Net-(J1-PadB8)
- J5 pad 9: (no net) -> Net-(J5-Pad9)
- L1 pad 1: Net-(C23-Pad1) -> Net-(C23-Pad2)
- L1 pad 2: Net-(C23-Pad2) -> Net-(C23-Pad1)
- L1 pad 3: Net-(C26-Pad2) -> Net-(C26-Pad1)
- L1 pad 4: Net-(C26-Pad1) -> Net-(C26-Pad2)
- RV1 pad 1: (no net) -> Net-(RV1-Pad1)
- T1 pad 1: Net-(C26-Pad1) -> Net-(D14-Pad2)
- T1 pad 2: Net-(D13-Pad2) -> GND
- T1 pad 3: GND -> Net-(D13-Pad2)
- T1 pad 4: Net-(D14-Pad2) -> Net-(T1-Pad4)
- T1 pad 5: (no net) -> Net-(C26-Pad1)
- U1 pad 10: (no net) -> Net-(U1-Pad10)
- U1 pad 11: (no net) -> Net-(U1-Pad11)
- U1 pad 17: (no net) -> Net-(U1-Pad17)
- U1 pad 18: (no net) -> Net-(U1-Pad18)
- U1 pad 19: (no net) -> Net-(U1-Pad19)
- U1 pad 20: (no net) -> Net-(U1-Pad20)
- U1 pad 21: (no net) -> Net-(U1-Pad21)
- U1 pad 22: (no net) -> Net-(U1-Pad22)
- U2 pad 15: (no net) -> Net-(U2-Pad15)
- U2 pad 16: (no net) -> Net-(U2-Pad16)
- U2 pad 2: (no net) -> Net-(U2-Pad2)
- U2 pad 4: (no net) -> Net-(U2-Pad4)
- U2 pad 5: (no net) -> Net-(U2-Pad5)
- U2 pad 6: (no net) -> Net-(U2-Pad6)
Routing:
- net +12V: track 2.07 -> 203.2 mm
- net +3V3: track 3.23 -> 137.2 mm, vias 0 -> 4
- net +5V: track 3.85 -> 96.1 mm, vias 0 -> 4
- net SCL: track 0.00 -> 63.6 mm, vias 0 -> 2
- net GND: track 8.48 -> 65.2 mm, vias 3 -> 87
- net SDA: track 0.00 -> 46.6 mm, vias 0 -> 2
- net ~INT: track 0.00 -> 40.2 mm, vias 0 -> 1
- net LOAD: track 48.3 -> 88.2 mm
- net RTS: track 0.00 -> 39.0 mm
- net TX: track 0.00 -> 37.3 mm, vias 0 -> 2
- net VCC: track 8.38 -> 40.8 mm
- net Net-(D7-Pad1): track 0.00 -> 31.1 mm, vias 0 -> 1
- net Net-(C5-Pad2): track 0.00 -> 28.8 mm, vias 0 -> 2
- net RX: track 0.00 -> 27.5 mm, vias 0 -> 2
- net Net-(D6-Pad2): track 0.00 -> 26.1 mm
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- added copper zone on B.Cu, net Earth
- added copper zone on F.Cu, net Earth
- added copper zone on B.Cu, net GND
- added copper zone on F.Cu, net GND
- added copper zone on F.Cu, net Net-(C26-Pad2)
Other:
- rule pad_to_mask_clearance: 0.051 -> 0
- board text added: "230V !!"
- board text added: "DATA"
- board text added: "E"
- board text added: "L"
- board text added: "N"
- board text removed: "230V"
- board text removed: "3V3"
- board text removed: "INT"
- board text removed: "LINE"
- board text removed: "NEUT"

Commit message: INA Begin
Other:
- board text added: "INT"
- board text removed: "ENA"
