File: NieuwOntwerp/Load.kicad_pcb (KiCad board)
At the start: 2 copper layers, 84 x 96 mm, 151 parts, among them J1 USB_C_Receptacle_USB2.0, J10 Conn_01x02, J2 Conn_01x02, J3 Conn_01x03, J4 Conn_01x02, J5 Conn_01x09_Male, J6 Conn_01x02, J7 Conn_01x03, J8 Conn_01x02, J9 Conn_01x02, Q1 Si2306, Q2 4809NG, Q3 IRF840, Q4 IRF840, Q5 IRF840, Q6 Si2306, T1 EE13, U1 ESP12E, U10 PC817, U11 TL431, U12 LM1117-3.3, U2 FT231XQ, U3 LM358, U4 MCP4725A0, U5 LM358, U6 INA219, U7 PCF8574, U8 SSD1306, U9 LNK364D

Commit message: Print_update
Parts:
- removed C5: 100uF, Capacitor_THT:CP_Radial_D5.0mm_P2.00mm
- removed D1: BZT52C-3V6, Diode_SMD:D_SOD-123
- removed D10, D9: MMSZ5225/3V, Diode_SMD:D_SOD-123
- removed D3: 1N4148, Diode2:DIO_LL4148
- removed D8: BZT52C-5V1, Diode_SMD:D_SOD-123
- removed J4, J8: Conn_01x02, Connector2:JST_XH_B2B-XH-AM_1x02_P2.50mm_Vertical
- removed Q1: Si2306, Package_TO_SOT_SMD:SOT-23
- removed R40, R41, R42, R45, R46, R55, R56: 10k, Resistor_SMD:R_0603_1608Metric
- removed R57: 1K2, Resistor_SMD:R_0603_1608Metric
- C1, C3: footprint Capacitor_SMD:C_0603_1608Metric -> Capacitor_SMD:C_0402_1005Metric
- C6: value 470pF -> 4,7nF
- J3, J7: value Conn_01x03 -> Din_02x03; footprint Connector2:JST_XH_B3B-XH-AM_1x03_P2.50mm_Vertical -> Connector_IDC:IDC-Header_2x03_P2.54mm_Vertical
- R1: value 330K -> 10K
- R2: value 10k -> 100K
- R20: value 100K -> 4K7
- R39: value 10k -> 0R; moved to F.Cu
- R4, R5: footprint Resistor_SMD:R_0603_1608Metric -> Resistor_SMD:R_0402_1005Metric
- R47: footprint Resistor_SMD:R_2512_6332Metric -> Resistor_THT:R_Axial_DIN0411_L9.9mm_D3.6mm_P5.08mm_Vertical
- R51: value 150 -> 1K2
- R54: value 6K8 -> 5K6
- R6: value 1K -> 10K
- R7: value 56K -> 27K
- RV1: footprint Potentiometer_THT:Potentiometer_Bourns_3266Y_Vertical -> Potentiometer_THT:Potentiometer_Bourns_3296W_Vertical
- U11: value TL431 -> TL432
- moved J9 139.8 mm to (190.4, 50.5), turned to 180 degrees
- moved C26 138.0 mm to (198.1, 94.6)
- moved F1 137.6 mm to (197.5, 65.9), turned to 90 degrees
- moved R47 135.6 mm to (193.8, 68.1)
- moved R1 135.1 mm to (171.6, 81.0), turned to 270 degrees
- moved R12 134.4 mm to (163.2, 63.6)
- moved D4 133.2 mm to (163.2, 61.8)
- moved R4 132.6 mm to (166.4, 55.7)
- moved C34 132.3 mm to (176.8, 70.4)
- moved C2 132.2 mm to (171.3, 55.7), turned to 270 degrees
- moved C1 132.0 mm to (167.6, 55.7)
- moved C21 132.0 mm to (163.2, 60.1)
- moved FB1 132.0 mm to (163.2, 54.9)
- moved J1 132.0 mm to (167.1, 47.3)
- moved U2 132.0 mm to (167.7, 60.3)
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Connections:
- C35 pad 2: +5V -> +12V
- C6 pad 1: Net-(C6-Pad1) -> GND
- H1 pad 1: GND -> Earth
- H2 pad 1: Net-(H2-Pad1) -> Earth
- J2 pad 4: Net-(D6-Pad2) -> Net-(J2-Pad4)
- J3 pad 1: /Front/SCL -> /Front/SDA
- J3 pad 3: /Front/SDA -> /Front/SCL
- J7 pad 1: SCL -> SDA
- J7 pad 2: ~INT -> Net-(J7-Pad2)
- J7 pad 3: SDA -> SCL
- Q3 pad 2: LOAD -> SHUNT
- Q4 pad 2: LOAD -> SHUNT
- Q5 pad 2: LOAD -> SHUNT
- R1 pad 1: LOAD -> RTS
- R1 pad 2: ADC -> +3V3
- R10 pad 2: +5V -> +12V
- R11 pad 1: Net-(C6-Pad1) -> GND
- R18 pad 2: +5V -> +12V
- R2 pad 1: ADC -> GND
- R2 pad 2: GND -> FAN_OVERRIDE
- R24 pad 1: Net-(D6-Pad2) -> Net-(J2-Pad4)
- R24 pad 2: +12V -> Net-(Q2-Pad1)
- R28 pad 1: SHUNT -> GND
- R31 pad 1: GND -> SHUNT
- R31 pad 2: SHUNT -> LOAD
- R32 pad 1: SHUNT -> GND
- R33 pad 2: SHUNT -> LOAD
- R34 pad 2: GND -> SHUNT
- R37 pad 1: SHUNT -> GND
- R38 pad 2: Net-(J3-Pad2) -> Net-(J3-Pad5)
- R39 pad 1: VDC -> Net-(C31-Pad2)
- R39 pad 2: Net-(J5-Pad1) -> Net-(R39-Pad2)
- R54 pad 1: Net-(C31-Pad2) -> Net-(R39-Pad2)
- R6 pad 1: Net-(D3-Pad1) -> GND
- R6 pad 2: Net-(C5-Pad2) -> Net-(R6-Pad2)
- R7 pad 2: Net-(C5-Pad2) -> THERM
- RV1 pad 2: +5V -> +12V
- U1 pad 10: Net-(U1-Pad10) -> Net-(R6-Pad2)
- U1 pad 2: ADC -> Net-(U1-Pad2)
- U1 pad 4: ~INT -> FAN_OVERRIDE
- U1 pad 6: FAN_OVERRIDE -> ~INT
- U5 pad 8: +5V -> +12V
- U7 pad 10: Net-(J5-Pad7) -> Net-(J5-Pad6)
- U7 pad 11: Net-(J5-Pad6) -> Net-(J5-Pad7)
- U7 pad 12: Net-(J5-Pad5) -> Net-(J5-Pad8)
- U7 pad 13: Net-(J3-Pad2) -> Net-(J3-Pad5)
- U7 pad 9: Net-(J5-Pad8) -> Net-(J5-Pad5)
Routing:
- net SHUNT: track 41.9 -> 186.8 mm
- net +5V: track 96.1 -> 0.00 mm, vias 4 -> 0
- net +12V: track 203.2 -> 113.9 mm, vias 0 -> 5
- net LOAD: track 88.2 -> 0.00 mm
- net Net-(J2-Pad4): track 0.00 -> 87.6 mm
- net +3V3: track 137.2 -> 54.3 mm, vias 4 -> 3
- net ~INT: track 40.2 -> 0.00 mm, vias 1 -> 0
- net Net-(J3-Pad2): track 38.0 -> 0.00 mm, vias 1 -> 0
- net VCC: track 40.8 -> 12.6 mm
- net Net-(C16-Pad2): track 0.00 -> 26.6 mm
- net Net-(J3-Pad5): track 0.00 -> 26.0 mm, vias 0 -> 1
- net ADC: track 26.0 -> 0.00 mm
- net Net-(C23-Pad2): track 0.00 -> 25.2 mm
- net Net-(R51-Pad1): track 23.5 -> 0.00 mm
- net FAN_OVERRIDE: track 23.2 -> 46.6 mm, vias 2 -> 3
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- removed copper zone on B.Cu, net GND
- removed copper zone on F.Cu, net GND
Other:
- outline, holes or cut-outs redrawn
- board text added: "1"
- board text added: "NC"
- board text removed: "230V !!"
- board text removed: "E"
- board text removed: "L"
- board text removed: "N"

Commit message: print update
Parts:
- moved R34 21.8 mm to (132.4, 98.4), turned to 180 degrees
- moved R31 20.0 mm to (133.1, 100.4), turned to 0 degrees
- moved C13 18.3 mm to (131.7, 96.0)
- moved U6 15.9 mm to (134.3, 95.5), turned to 270 degrees
- moved R33 13.9 mm to (135.4, 98.4)
- moved C9 12.3 mm to (136.9, 96.0), turned to 90 degrees
- moved R20 11.2 mm to (146.4, 62.4)
- moved R9 8.83 mm to (147.0, 88.5), turned to 90 degrees
- moved R2 8.41 mm to (140.2, 80.8), turned to 0 degrees
- moved D7 8.05 mm to (147.9, 59.0)
- moved R50 7.48 mm to (167.9, 93.0)
- moved C7 7.44 mm to (130.6, 89.6)
- moved R26 7.30 mm to (130.6, 88.0)
- moved R8 5.68 mm to (145.4, 88.5)
- moved U4 5.66 mm to (143.8, 91.9)
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Connections:
- J1 pad A5: Net-(J1-PadA5) -> (no net)
- J1 pad A8: Net-(J1-PadA8) -> (no net)
- J1 pad B5: Net-(J1-PadB5) -> (no net)
- J1 pad B8: Net-(J1-PadB8) -> (no net)
- J3 pad 2: Net-(J3-Pad2) -> (no net)
- J5 pad 9: Net-(J5-Pad9) -> (no net)
- J7 pad 2: Net-(J7-Pad2) -> (no net)
- RV1 pad 1: Net-(RV1-Pad1) -> (no net)
- T1 pad 4: Net-(T1-Pad4) -> (no net)
- U1 pad 11: Net-(U1-Pad11) -> (no net)
- U1 pad 17: Net-(U1-Pad17) -> (no net)
- U1 pad 18: Net-(U1-Pad18) -> (no net)
- U1 pad 19: Net-(U1-Pad19) -> (no net)
- U1 pad 2: Net-(U1-Pad2) -> (no net)
- U1 pad 20: Net-(U1-Pad20) -> (no net)
- U1 pad 21: Net-(U1-Pad21) -> (no net)
- U1 pad 22: Net-(U1-Pad22) -> (no net)
- U2 pad 15: Net-(U2-Pad15) -> (no net)
- U2 pad 16: Net-(U2-Pad16) -> (no net)
- U2 pad 2: Net-(U2-Pad2) -> (no net)
- U2 pad 4: Net-(U2-Pad4) -> (no net)
- U2 pad 5: Net-(U2-Pad5) -> (no net)
- U2 pad 6: Net-(U2-Pad6) -> (no net)
- U5 pad 1: Net-(R17-Pad1) -> Net-(R25-Pad1)
- U5 pad 2: Net-(R16-Pad2) -> Net-(R23-Pad2)
- U5 pad 3: Net-(U4-Pad1) -> Net-(R21-Pad1)
- U5 pad 5: Net-(R21-Pad1) -> Net-(U4-Pad1)
- U5 pad 6: Net-(R23-Pad2) -> Net-(R16-Pad2)
- U5 pad 7: Net-(R25-Pad1) -> Net-(R17-Pad1)
Routing:
- net SHUNT: track 186.8 -> 55.6 mm
- net Net-(J2-Pad4): track 87.6 -> 6.86 mm
- net +12V: track 113.9 -> 39.9 mm, vias 5 -> 2
- net Net-(J5-Pad5): track 60.7 -> 24.1 mm
- net FAN_OVERRIDE: track 46.6 -> 11.9 mm, vias 3 -> 0
- net ~INT: track 0.00 -> 29.5 mm, vias 0 -> 1
- net +3V3: track 54.3 -> 28.3 mm, vias 3 -> 2
- net SDA: track 31.1 -> 53.8 mm, vias 2 -> 1
- net Net-(U1-Pad2): track 20.5 -> 0.00 mm
- net Net-(C5-Pad2): track 15.4 -> 0.00 mm, vias 2 -> 0
- net FAN_TACH: track 13.9 -> 27.3 mm
- net Net-(R21-Pad1): track 16.5 -> 5.62 mm, vias 2 -> 0
- net Net-(R6-Pad2): track 0.00 -> 10.7 mm
- net (no net): track 0.00 -> 10.2 mm
- net THERM: track 89.9 -> 79.7 mm
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
Commit message: Print gereed
Parts:
- moved C35 11.9 mm to (151.8, 98.0)
- moved C31 5.66 mm to (160.9, 95.2)
- moved C32 5.62 mm to (155.4, 97.7), turned to 90 degrees
- moved U12 4.93 mm to (149.9, 103.2)
- moved R51 3.94 mm to (160.9, 93.5), turned to 0 degrees
- moved L2 3.41 mm to (157.6, 100.7)
- moved C33 3.13 mm to (155.2, 103.5), turned to 270 degrees
- moved R53 3.00 mm to (158.8, 94.3), turned to 270 degrees
- moved R54 2.61 mm to (157.6, 104.3)
- moved U11 2.26 mm to (159.9, 97.7), turned to 270 degrees
- moved R39 0.72 mm to (157.6, 102.8)
- moved C30 0.63 mm to (164.1, 93.5)
- moved R50 0.60 mm to (167.9, 93.5)
- moved D14 0.47 mm to (166.8, 96.5)
- moved C29 0.29 mm to (165.0, 101.2)
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Routing:
- net +3V3: track 28.3 -> 175.3 mm, vias 2 -> 10
- net +12V: track 39.9 -> 130.6 mm, vias 2 -> 6
- net GND: track 55.3 -> 86.5 mm, vias 41 -> 67
- net SDA: track 53.8 -> 78.0 mm, vias 1 -> 2
- net SCL: track 50.1 -> 73.1 mm, vias 1 -> 2
- net FAN_OVERRIDE: track 11.9 -> 31.6 mm
- net Net-(R51-Pad1): track 5.63 -> 21.5 mm
- net Net-(C31-Pad1): track 7.08 -> 22.9 mm
- net (no net): track 10.2 -> 0.00 mm
- net Net-(C31-Pad2): track 0.00 -> 9.84 mm
- net Net-(C29-Pad1): track 8.70 -> 15.9 mm
- net Net-(J5-Pad1): track 28.4 -> 24.9 mm
- net Net-(J5-Pad2): track 30.6 -> 27.2 mm
- net THERM: track 79.7 -> 76.6 mm, vias 0 -> 1
- net TX: track 34.8 -> 37.8 mm
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- added copper zone on B.Cu, net GND
- added copper zone on F.Cu, net GND
Other:
- net class Default: clearance 0.2 -> 0.15; trace_width 0.25 -> 0.152; via_dia 0.8 -> 0.5; via_drill 0.4 -> 0.3
- rule trace_clearance: 0.2 -> 0.15
- rule trace_min: 0.1016 -> 0.15
- rule via_min_size: 0.3048 -> 0.4
- board text added: "+"
- board text added: "+12V"
- board text added: "+3.3V"
- board text added: "-"
- board text added: "."
- board text added: "0V"
- board text added: "230V!"
- board text added: "E"
- board text added: "L"
- board text added: "N"
- board text added: "PWM"
- board text removed: "DATA"
- board text removed: "INT"
- board text removed: "NC"

Commit message: 21-11-2021
Parts:
- U6: value INA219 -> INA219AxDCN
- moved C13 5.25 mm to (136.9, 96.0)
- moved C9 5.20 mm to (131.7, 96.0)
- moved U6 0.11 mm to (134.3, 95.4), turned to 90 degrees
- turned R33 to 0 degrees
Connections:
- J1 pad A5: (no net) -> Net-(J1-PadA5)
- J1 pad A8: (no net) -> Net-(J1-PadA8)
- J1 pad B5: (no net) -> Net-(J1-PadB5)
- J1 pad B8: (no net) -> Net-(J1-PadB8)
- J3 pad 2: (no net) -> Net-(J3-Pad2)
- J5 pad 9: (no net) -> Net-(J5-Pad9)
- J7 pad 2: (no net) -> Net-(J7-Pad2)
- RV1 pad 1: (no net) -> Net-(RV1-Pad1)
- T1 pad 4: (no net) -> Net-(T1-Pad4)
- U1 pad 11: (no net) -> Net-(U1-Pad11)
- U1 pad 17: (no net) -> Net-(U1-Pad17)
- U1 pad 18: (no net) -> Net-(U1-Pad18)
- U1 pad 19: (no net) -> Net-(U1-Pad19)
- U1 pad 2: (no net) -> Net-(U1-Pad2)
- U1 pad 20: (no net) -> Net-(U1-Pad20)
- U1 pad 21: (no net) -> Net-(U1-Pad21)
- U1 pad 22: (no net) -> Net-(U1-Pad22)
- U2 pad 15: (no net) -> Net-(U2-Pad15)
- U2 pad 16: (no net) -> Net-(U2-Pad16)
- U2 pad 2: (no net) -> Net-(U2-Pad2)
- U2 pad 4: (no net) -> Net-(U2-Pad4)
- U2 pad 5: (no net) -> Net-(U2-Pad5)
- U2 pad 6: (no net) -> Net-(U2-Pad6)
- U6 pad 1: GND -> Net-(C9-Pad1)
- U6 pad 2: GND -> Net-(C9-Pad2)
- U6 pad 3: SDA -> GND
- U6 pad 4: SCL -> +3V3
- U6 pad 5: +3V3 -> SCL
- U6 pad 6: GND -> SDA
- U6 pad 7: Net-(C9-Pad2) -> GND
- U6 pad 8: Net-(C9-Pad1) -> GND
Routing:
- net +3V3: track 175.3 -> 168.0 mm
- net Net-(C9-Pad1): track 3.49 -> 6.18 mm
- net GND: track 86.5 -> 88.9 mm
- net SCL: track 73.1 -> 71.3 mm
- net LOAD: track 6.40 -> 7.12 mm
- net SDA: track 78.0 -> 77.9 mm, vias 2 -> 4
Other:
- outline, holes or cut-outs redrawn
- net class Default: via_dia 0.5 -> 0.6
- rule via_min_drill: 0.2 -> 0.3
