File: NieuwOntwerp/Front.sch (KiCad schematic (older format))
At the start: 27 parts, among them J6 Conn_01x03, J7 Conn_01x02, SW1 Switch_6x6_SMT, SW2 Switch_6x6_SMT, SW3 Switch_6x6_SMT, SW4 Switch_6x6_SMT, U8 SSD1306, U9 PCF8574

Commit message: Sync_21-04-27
Parts:
- added J3: Conn_01x09_Male, Connector_PinHeader_2.54mm:PinHeader_1x09_P2.54mm_Vertical, symbol Connector:Conn_01x09_Male
- added J4, J8: Conn_01x02, Connector2:JST_XH_B2B-XH-AM_1x02_P2.50mm_Vertical, symbol Connector_Generic:Conn_01x02
- added J5: Conn_01x03, Connector2:JST_XH_B3B-XH-AM_1x03_P2.50mm_Vertical, symbol Connector_Generic:Conn_01x03
- added J9: Conn_01x02, Connector2:JST_XH_B3B-XH-AM_1x03_P2.50mm_Vertical, symbol Connector_Generic:Conn_01x03
- R24, R25, R26, R27, R28, R29, R30, R31, R32: footprint Resistor_SMD:R_0603_1608Metric_Pad1.05x0.95mm_HandSolder -> Resistor_SMD:R_0603_1608Metric
Connections:
- net SCL: now also J5.1 (Pin_1)
- net SDA: now also J5.3 (Pin_3)
- new net +3V3: J8.1 (Pin_1)
- new net Earth: J9.2 (Pin_2)
- new net GND: J4.2 (Pin_2), J8.2 (Pin_2)
- new net LINE: J9.1 (Pin_1)
- new net LOAD: J4.1 (Pin_1)
- new net NEUTRAL: J9.3 (Pin_3)
- new net ~INT: J5.2 (Pin_2)
Other:
- note added: "230V AC"
- note added: "Connections to case"
- note added: "Connectors to Front Panel"
- note added: "Front"
- note added: "Mounting"
- moved on the sheet: C21, C22, D5, D6, D7, D8, H10, H11, H12, H9, J6, J7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

Commit message: 2021-05-13_01
Parts:
- removed D5, D6, D7, D8: LED, LED_SMD:LED_0603_1608Metric_Pad1.05x0.95mm_HandSolder, symbol Device:LED
- removed R28, R29, R30, R31: 270R, Resistor_SMD:R_0603_1608Metric, symbol Device:R
- removed SW1, SW2, SW3, SW4: Switch_6x6_SMT, Switches:SW_SPST_6x6x20mm_SMD, symbol OPL-Switch:Switch_6x6_SMT
- added R? (x4): 10k, Resistor_SMD:R_0603_1608Metric, symbol Device:R
- renumbered C21 to C11, C22 to C12, H9 to H5, H10 to H6, H11 to H7, H12 to H8, J6 to J3, J7 to J4, J3 to J5, J4 to J6, J5 to J7, R32 to R38, R24 to R39, R25 to R40, R26 to R41, R27 to R42, U9 to U7
Connections:
- net VDC: now also R?.1, R?.1, R?.1, R?.1
- net at U7.10 (P5): now also J5.7 (Pin_7), R?.2
- net at U7.11 (P6): now also J5.6 (Pin_6), R?.2
- net at U7.12 (P7): now also J5.5 (Pin_5), R?.2
- net at R39.2, U7.4 (P0): now also J5.1 (Pin_1)
- net at R40.2, U7.5 (P1): now also J5.2 (Pin_2)
- net at R41.2, U7.6 (P2): now also J5.3 (Pin_3)
- net at R42.2, U7.7 (P3): now also J5.4 (Pin_4)
- net at U7.9 (P4): now also J5.8 (Pin_8), R?.2
- no-connect marks 0 -> 1
Other:
- note removed: "DOWN"
- note removed: "LEFT"
- note removed: "RIGHT"
- note removed: "UP"
- moved on the sheet: C11, C12, J5, R39, R40, R41, R42

Commit message: 2021-05-14_02
Parts:
- removed J7: Conn_01x03, Connector2:JST_XH_B3B-XH-AM_1x03_P2.50mm_Vertical, symbol Connector_Generic:Conn_01x03
- removed J8: Conn_01x02, Connector2:JST_XH_B2B-XH-AM_1x02_P2.50mm_Vertical, symbol Connector_Generic:Conn_01x02
- gave numbers to parts that had none: 4
Other:
- note removed: "Connectors to Front Panel"
Changed lines of the file:
@@
-	1    0    0    -1
-$EndComp
-$Comp
-L power:GNDA #PWR042
-U 1 1 60370CB6
-P 3100 2800
-F 0 "#PWR042" H 3100 2550 50  0001 C CNN
-F 1 "GNDA" H 3105 2627 50  0000 C CNN
-F 2 "" H 3100 2800 50  0001 C CNN
-F 3 "" H 3100 2800 50  0001 C CNN
-	1    3100 2800
 	1    0    0    -1
 $EndComp
@@
 Text Notes 950  1000 0    50   ~ 0
 Front
-Wire Notes Line
-	10000 3450 8550 3450
 Text Notes 5950 2550 0    50   ~ 0
 Mounting
@@
 	-1   0    0    -1
 $EndComp
-$Comp
-L power:GND #PWR?
-U 1 1 607060D9
-P 8950 1500
-AR Path="/607060D9" Ref="#PWR?"  Part="1"
-AR Path="/60357CC4/607060D9" Ref="#PWR049"  Part="1"
-F 0 "#PWR049" H 8950 1250 50  0001 C CNN
-F 1 "GND" H 8955 1327 50  0000 C CNN
-F 2 "" H 8950 1500 50  0001 C CNN
-F 3 "" H 8950 1500 50  0001 C CNN
-	1    8950 1500
-	1    0    0    -1
-$EndComp
 Text GLabel 8950 1400 2    50   Input ~ 0
 LOAD
@@
 $EndComp
 $Comp
-L Connector_Generic:Conn_01x03 J?
-U 1 1 607060F8
-P 8950 2600
-AR Path="/607060F8" Ref="J?"  Part="1"
-AR Path="/60357CC4/607060F8" Ref="J7"  Part="1"
-F 0 "J7" H 9150 2600 50  0000 C CNN
-F 1 "Conn_01x03" H 8868 2826 50  0000 C CNN
-F 2 "Connector2:JST_XH_B3B-XH-AM_1x03_P2.50mm_Vertical" H 8950 2600 50  0001 C CNN
-F 3 "~" H 8950 2600 50  0001 C CNN
-	1    8950 2600
-	-1   0    0    -1
-$EndComp
-$Comp
-L Connector_Generic:Conn_01x02 J?
-U 1 1 607060FE
-P 8950 3050
-AR Path="/607060FE" Ref="J?"  Part="1"
-AR Path="/60357CC4/607060FE" Ref="J8"  Part="1"
-F 0 "J8" H 9150 3000 50  0000 C CNN
-F 1 "Conn_01x02" H 8868 3176 50  0000 C CNN
-F 2 "Connector2:JST_XH_B2B-XH-AM_1x02_P2.50mm_Vertical" H 8950 3050 50  0001 C CNN
-F 3 "~" H 8950 3050 50  0001 C CNN
-	1    8950 3050
-	-1   0    0    -1
-$EndComp
-Wire Wire Line
-	9150 3050 9400 3050
-Wire Wire Line
-	9150 3150 9400 3150
-Wire Wire Line
-	9150 2500 9350 2500
-Wire Wire Line
-	9150 2700 9350 2700
-Wire Wire Line
-	9150 2600 9600 2600
-Text GLabel 9350 2500 2    50   Input ~ 0
-SCL
-Text GLabel 9350 2700 2    50   Input ~ 0
-SDA
-$Comp
-L power:+3.3V #PWR?
-U 1 1 6070610B
-P 9400 3050
-AR Path="/6070610B" Ref="#PWR?"  Part="1"
-AR Path="/60357CC4/6070610B" Ref="#PWR050"  Part="1"
-F 0 "#PWR050" H 9400 2900 50  0001 C CNN
-F 1 "+3.3V" H 9415 3223 50  0000 C CNN
-F 2 "" H 9400 3050 50  0001 C CNN
-F 3 "" H 9400 3050 50  0001 C CNN
-	1    9400 3050
-	1    0    0    -1
-$EndComp
-$Comp
-L power:GND #PWR?
-U 1 1 60706111
-P 9400 3150
-AR Path="/60706111" Ref="#PWR?"  Part="1"
-AR Path="/60357CC4/60706111" Ref="#PWR051"  Part="1"
-F 0 "#PWR051" H 9400 2900 50  0001 C CNN
-F 1 "GND" H 9405 2977 50  0000 C CNN
-F 2 "" H 9400 3150 50  0001 C CNN
-F 3 "" H 9400 3150 50  0001 C CNN
-	1    9400 3150
-	1    0    0    -1
-$EndComp
-Wire Notes Line
-	8550 2200 10000 2200
-Wire Notes Line
-	10000 2200 10000 3450
-Wire Notes Line
-	8550 3450 8550 2200
-Text Notes 8600 2300 0    50   ~ 0
-Connectors to Front Panel
-Text GLabel 9600 2600 2    50   Input ~ 0
-~INT
-$Comp
 L Connector:Conn_01x09_Male J5
 U 1 1 608A7010
@@
 P 3800 1300
 AR Path="/60AAA1E7" Ref="R?"  Part="1"
-AR Path="/60357CC4/60AAA1E7" Ref="R?"  Part="1"
-F 0 "R?" H 3750 1500 50  0000 L CNN
+AR Path="/60357CC4/60AAA1E7" Ref="R45"  Part="1"
+F 0 "R45" H 3750 1500 50  0000 L CNN
 F 1 "10k" V 3800 1200 50  0000 L CNN
 F 2 "Resistor_SMD:R_0603_1608Metric" V 3730 1300 50  0001 C CNN
@@
 P 3950 1300
 AR Path="/60AAA1ED" Ref="R?"  Part="1"
-AR Path="/60357CC4/60AAA1ED" Ref="R?"  Part="1"
-F 0 "R?" H 3900 1500 50  0000 L CNN
+AR Path="/60357CC4/60AAA1ED" Ref="R46"  Part="1"
+F 0 "R46" H 3900 1500 50  0000 L CNN
 F 1 "10k" V 3950 1200 50  0000 L CNN
 F 2 "Resistor_SMD:R_0603_1608Metric" V 3880 1300 50  0001 C CNN
@@
 P 4100 1300
 AR Path="/60AAA1F3" Ref="R?"  Part="1"
-AR Path="/60357CC4/60AAA1F3" Ref="R?"  Part="1"
-F 0 "R?" H 4050 1500 50  0000 L CNN
+AR Path="/60357CC4/60AAA1F3" Ref="R55"  Part="1"
+F 0 "R55" H 4050 1500 50  0000 L CNN
 F 1 "10k" V 4100 1200 50  0000 L CNN
 F 2 "Resistor_SMD:R_0603_1608Metric" V 4030 1300 50  0001 C CNN
@@
 P 4250 1300
 AR Path="/60AAA1F9" Ref="R?"  Part="1"
-AR Path="/60357CC4/60AAA1F9" Ref="R?"  Part="1"
-F 0 "R?" H 4200 1500 50  0000 L CNN
+AR Path="/60357CC4/60AAA1F9" Ref="R56"  Part="1"
+F 0 "R56" H 4200 1500 50  0000 L CNN
 F 1 "10k" V 4250 1200 50  0000 L CNN
 F 2 "Resistor_SMD:R_0603_1608Metric" V 4180 1300 50  0001 C CNN
@@
 Connection ~ 3800 1900
 NoConn ~ 4500 2300
+$Comp
+L power:GND #PWR0103
+U 1 1 60A05EBE
+P 8950 1500
+F 0 "#PWR0103" H 8950 1250 50  0001 C CNN
+F 1 "GND" H 8955 1327 50  0000 C CNN
+F 2 "" H 8950 1500 50  0001 C CNN
+F 3 "" H 8950 1500 50  0001 C CNN
+	1    8950 1500
+	1    0    0    -1
+$EndComp
 $EndSCHEMATC

Commit message: start
Other:
- note added: "Address 0x3C"
- note added: "Address 0x40"
- note removed: "Address 0x38"
- note removed: "Address 0x78"
Changed lines of the file:
@@
 	6100 1300 6400 1300
 Text Notes 6300 1800 0    50   ~ 0
-Address 0x78
+Address 0x3C
 $Comp
 L power:VDC #PWR040
@@
 	5900 2350 5900 900
 Text Notes 1900 1250 0    50   ~ 0
-Address 0x38
+Address 0x40
 $Comp
 L Device:R R?

Commit message: Keyboard
Parts:
- removed R39, R40, R41, R42, R45, R46, R55, R56: 10k, Resistor_SMD:R_0603_1608Metric, symbol Device:R
Connections:
- net at U7.10 (P5): now also J5.6 (Pin_6); no longer J5.7 (Pin_7)
- net at U7.11 (P6): now also J5.7 (Pin_7); no longer J5.6 (Pin_6)
- net at U7.12 (P7): now also J5.8 (Pin_8); no longer J5.5 (Pin_5)
- net at U7.9 (P4): now also J5.5 (Pin_5); no longer J5.8 (Pin_8)
Other:
- moved on the sheet: J5
Changed lines of the file:
@@
 $EndDescr
-$Comp
-L Interface_Expansion:PCF8574 U?
-U 1 1 6035A425
-P 2650 1900
-AR Path="/6035A425" Ref="U?"  Part="1"
-AR Path="/60357CC4/6035A425" Ref="U7"  Part="1"
-F 0 "U7" H 2650 1950 50  0000 C CNN
-F 1 "PCF8574" H 2650 2050 50  0000 C CNN
-F 2 "Package_SO:SOIC-16W_7.5x10.3mm_P1.27mm" H 2650 1900 50  0001 C CNN
-F 3 "http://www.nxp.com/documents/data_sheet/PCF8574_PCF8574A.pdf" H 2650 1900 50  0001 C CNN
-	1    2650 1900
-	1    0    0    -1
-$EndComp
-$Comp
-L Device:R R?
-U 1 1 6035A437
-P 3200 1300
-AR Path="/6035A437" Ref="R?"  Part="1"
-AR Path="/60357CC4/6035A437" Ref="R39"  Part="1"
-F 0 "R39" H 3150 1500 50  0000 L CNN
-F 1 "10k" V 3200 1200 50  0000 L CNN
-F 2 "Resistor_SMD:R_0603_1608Metric" V 3130 1300 50  0001 C CNN
-F 3 "~" H 3200 1300 50  0001 C CNN
-	1    3200 1300
-	1    0    0    -1
-$EndComp
-$Comp
-L Device:R R?
-U 1 1 6035A43D
-P 3350 1300
-AR Path="/6035A43D" Ref="R?"  Part="1"
-AR Path="/60357CC4/6035A43D" Ref="R40"  Part="1"
-F 0 "R40" H 3300 1500 50  0000 L CNN
-F 1 "10k" V 3350 1200 50  0000 L CNN
-F 2 "Resistor_SMD:R_0603_1608Metric" V 3280 1300 50  0001 C CNN
-F 3 "~" H 3350 1300 50  0001 C CNN
-	1    3350 1300
-	1    0    0    -1
-$EndComp
-$Comp
-L Device:R R?
-U 1 1 6035A443
-P 3500 1300
-AR Path="/6035A443" Ref="R?"  Part="1"
-AR Path="/60357CC4/6035A443" Ref="R41"  Part="1"
-F 0 "R41" H 3450 1500 50  0000 L CNN
-F 1 "10k" V 3500 1200 50  0000 L CNN
-F 2 "Resistor_SMD:R_0603_1608Metric" V 3430 1300 50  0001 C CNN
-F 3 "~" H 3500 1300 50  0001 C CNN
-	1    3500 1300
-	1    0    0    -1
-$EndComp
-$Comp
-L Device:R R?
-U 1 1 6035A449
-P 3650 1300
-AR Path="/6035A449" Ref="R?"  Part="1"
-AR Path="/60357CC4/6035A449" Ref="R42"  Part="1"
-F 0 "R42" H 3600 1500 50  0000 L CNN
-F 1 "10k" V 3650 1200 50  0000 L CNN
-F 2 "Resistor_SMD:R_0603_1608Metric" V 3580 1300 50  0001 C CNN
-F 3 "~" H 3650 1300 50  0001 C CNN
-	1    3650 1300
-	1    0    0    -1
-$EndComp
-Wire Wire Line
-	3200 1150 3350 1150
 $Comp
 L Connector_Generic:Conn_01x03 J?
@@
 $EndComp
 $Comp
-L power:VDC #PWR043
-U 1 1 6036BD27
-P 3050 1150
-F 0 "#PWR043" H 3050 1050 50  0001 C CNN
-F 1 "VDC" H 3065 1323 50  0000 C CNN
-F 2 "" H 3050 1150 50  0001 C CNN
-F 3 "" H 3050 1150 50  0001 C CNN
-	1    3050 1150
-	1    0    0    -1
-$EndComp
-$Comp
 L power:VDC #PWR047
 U 1 1 6036C1FE
@@
 Wire Wire Line
 	1300 1650 1500 1650
-Wire Wire Line
-	2150 1800 2150 1900
-Connection ~ 2150 1900
-Wire Wire Line
-	2150 1900 2150 2000
 Wire Wire Line
 	1300 1550 1750 1550
@@
 AR Path="/601A616F" Ref="R?"  Part="1"
 AR Path="/60357CC4/601A616F" Ref="R38"  Part="1"
-F 0 "R38" H 1950 2200 50  0000 L CNN
+F 0 "R38" H 1900 2300 50  0000 L CNN
 F 1 "10k" V 1900 2050 50  0000 L CNN
 F 2 "Resistor_SMD:R_0603_1608Metric" V 1830 2150 50  0001 C CNN
@@
 	1    0    0    -1
 $EndComp
-Connection ~ 2150 2000
 Connection ~ 1150 2550
 Wire Notes Line
@@
 L Connector:Conn_01x09_Male J5
 U 1 1 608A7010
-P 4700 1900
-F 0 "J5" H 4850 2550 50  0000 C CNN
-F 1 "Conn_01x09_Male" H 4700 2450 50  0000 C CNN
-F 2 "Connector_PinHeader_2.54mm:PinHeader_1x09_P2.54mm_Vertical" H 4700 1900 50  0001 C CNN
-F 3 "~" H 4700 1900 50  0001 C CNN
-	1    4700 1900
+P 3500 1900
+F 0 "J5" H 3650 2550 50  0000 C CNN
+F 1 "Conn_01x09_Male" H 3500 2450 50  0000 C CNN
+F 2 "Connector_PinHeader_2.54mm:PinHeader_1x09_P2.54mm_Vertical" H 3500 1900 50  0001 C CNN
+F 3 "~" H 3500 1900 50  0001 C CNN
+	1    3500 1900
 	-1   0    0    -1
 $EndComp
-Connection ~ 3350 1150
-Connection ~ 3500 1150
-Wire Wire Line
-	3500 1150 3650 1150
-Wire Wire Line
-	3350 1150 3500 1150
-$Comp
-L Device:R R?
-U 1 1 60AAA1E7
-P 3800 1300
-AR Path="/60AAA1E7" Ref="R?"  Part="1"
-AR Path="/60357CC4/60AAA1E7" Ref="R45"  Part="1"
-F 0 "R45" H 3750 1500 50  0000 L CNN
-F 1 "10k" V 3800 1200 50  0000 L CNN
-F 2 "Resistor_SMD:R_0603_1608Metric" V 3730 1300 50  0001 C CNN
-F 3 "~" H 3800 1300 50  0001 C CNN
-	1    3800 1300
-	1    0    0    -1
-$EndComp
-$Comp
-L Device:R R?
-U 1 1 60AAA1ED
-P 3950 1300
-AR Path="/60AAA1ED" Ref="R?"  Part="1"
-AR Path="/60357CC4/60AAA1ED" Ref="R46"  Part="1"
-F 0 "R46" H 3900 1500 50  0000 L CNN
-F 1 "10k" V 3950 1200 50  0000 L CNN
-F 2 "Resistor_SMD:R_0603_1608Metric" V 3880 1300 50  0001 C CNN
-F 3 "~" H 3950 1300 50  0001 C CNN
-	1    3950 1300
-	1    0    0    -1
-$EndComp
-$Comp
-L Device:R R?
-U 1 1 60AAA1F3
-P 4100 1300
-AR Path="/60AAA1F3" Ref="R?"  Part="1"
-AR Path="/60357CC4/60AAA1F3" Ref="R55"  Part="1"
-F 0 "R55" H 4050 1500 50  0000 L CNN
-F 1 "10k" V 4100 1200 50  0000 L CNN
-F 2 "Resistor_SMD:R_0603_1608Metric" V 4030 1300 50  0001 C CNN
-F 3 "~" H 4100 1300 50  0001 C CNN
-	1    4100 1300
-	1    0    0    -1
-$EndComp
-$Comp
-L Device:R R?
-U 1 1 60AAA1F9
-P 4250 1300
-AR Path="/60AAA1F9" Ref="R?"  Part="1"
-AR Path="/60357CC4/60AAA1F9" Ref="R56"  Part="1"
-F 0 "R56" H 4200 1500 50  0000 L CNN
-F 1 "10k" V 4250 1200 50  0000 L CNN
-F 2 "Resistor_SMD:R_0603_1608Metric" V 4180 1300 50  0001 C CNN
-F 3 "~" H 4250 1300 50  0001 C CNN
-	1    4250 1300
-	1    0    0    -1
-$EndComp
-Wire Wire Line
-	3650 1150 3800 1150
-Connection ~ 3650 1150
-Connection ~ 3800 1150
-Wire Wire Line
-	3800 1150 3950 1150
-Connection ~ 3950 1150
-Wire Wire Line
-	3950 1150 4100 1150
-Connection ~ 4100 1150
-Wire Wire Line
-	4100 1150 4250 1150
-Wire Wire Line
-	3050 1150 3200 1150
-Connection ~ 3200 1150
-Wire Wire Line
-	3150 1500 3200 1500
-Wire Wire Line
-	3200 1500 3200 1450
-Wire Wire Line
-	3150 1600 3350 1600
-Wire Wire Line
-	3350 1600 3350 1450
-Wire Wire Line
-	3150 1700 3500 1700
-Wire Wire Line
-	3500 1700 3500 1450
-Wire Wire Line
-	3150 1800 3650 1800
-Wire Wire Line
-	3650 1800 3650 1450
-Wire Wire Line
-	3150 1900 3800 1900
-Wire Wire Line
-	3800 1900 3800 1450
-Wire Wire Line
-	3150 2000 3950 2000
-Wire Wire Line
-	3950 2000 3950 1450
-Wire Wire Line
-	3150 2100 4100 2100
-Wire Wire Line
-	4100 2100 4100 2000
-Wire Wire Line
-	3150 2200 4250 2200
-Wire Wire Line
-	4250 2200 4250 1900
-Wire Wire Line
-	3200 1500 4500 1500
-Connection ~ 3200 1500
-Wire Wire Line
-	3350 1600 4500 1600
-Connection ~ 3350 1600
-Wire Wire Line
-	3500 1700 4500 1700
-Connection ~ 3500 1700
-Wire Wire Line
-	3650 1800 4500 1800
-Connection ~ 3650 1800
-Wire Wire Line
-	4250 1900 4500 1900
-Connection ~ 4250 1900
-Wire Wire Line
-	4250 1900 4250 1450
-Wire Wire Line
-	4100 2000 4500 2000
-Connection ~ 4100 2000
-Wire Wire Line
-	4100 2000 4100 1450
-Wire Wire Line
-	3950 2000 3950 2300
-Wire Wire Line
-	3950 2300 4350 2300
-Wire Wire Line
-	4350 2300 4350 2100
-Wire Wire Line
-	4350 2100 4500 2100
-Connection ~ 3950 2000
-Wire Wire Line
-	3800 1900 3800 2400
-Wire Wire Line
-	3800 2400 4450 2400
-Wire Wire Line
-	4450 2400 4450 2200
-Wire Wire Line
-	4450 2200 4500 2200
-Connection ~ 3800 1900
-NoConn ~ 4500 2300
+NoConn ~ 3300 2300
 $Comp
 L power:GND #PWR0103
@@
 	1    0    0    -1
 $EndComp
+Connection ~ 2150 2000
+Wire Wire Line
+	2150 1900 2150 2000
+Wire Wire Line
+	2150 1800 2150 1900
+Connection ~ 2150 1900
+$Comp
+L Interface_Expansion:PCF8574 U?
+U 1 1 6035A425
+P 2650 1900
+AR Path="/6035A425" Ref="U?"  Part="1"
+AR Path="/60357CC4/6035A425" Ref="U7"  Part="1"
+F 0 "U7" H 2650 1950 50  0000 C CNN
+F 1 "PCF8574" H 2650 2050 50  0000 C CNN
+F 2 "Package_SO:SOIC-16W_7.5x10.3mm_P1.27mm" H 2650 1900 50  0001 C CNN
+F 3 "http://www.nxp.com/documents/data_sheet/PCF8574_PCF8574A.pdf" H 2650 1900 50  0001 C CNN
+	1    2650 1900
+	1    0    0    -1
+$EndComp
+Wire Wire Line
+	3150 1500 3300 1500
+Wire Wire Line
+	3150 1600 3300 1600
+Wire Wire Line
+	3150 1700 3300 1700
+Wire Wire Line
+	3150 1800 3300 1800
+Wire Wire Line
+	3150 1900 3300 1900
+Wire Wire Line
+	3150 2000 3300 2000
+Wire Wire Line
+	3150 2100 3300 2100
+Wire Wire Line
+	3150 2200 3300 2200
 $EndSCHEMATC

Commit message: Print_update
Parts:
- removed J3: Conn_01x03, Connector2:JST_XH_B3B-XH-AM_1x03_P2.50mm_Vertical, symbol Connector_Generic:Conn_01x03
- removed J4: Conn_01x02, Connector2:JST_XH_B2B-XH-AM_1x02_P2.50mm_Vertical, symbol Connector_Generic:Conn_01x02
- added J3: Din_02x03, Connector_IDC:IDC-Header_2x03_P2.54mm_Vertical, symbol Connector_Generic:Conn_02x03_Odd_Even
Connections:
- net GNDA: now also J3.6 (Pin_6)
- net SCL: now also J3.3 (Pin_3)
- net SDA: now also J3.1 (Pin_1)
- net VDC: now also J3.4 (Pin_4)
- net at R38.2, U7.13 (~INT~): now also J3.5 (Pin_5)
- no-connect marks 1 -> 2
Changed lines of the file:
@@
 $EndDescr
-$Comp
-L Connector_Generic:Conn_01x03 J?
-U 1 1 6035A4F2
-P 1100 1550
-AR Path="/6035A4F2" Ref="J?"  Part="1"
-AR Path="/60357CC4/6035A4F2" Ref="J3"  Part="1"
-F 0 "J3" H 1018 1867 50  0000 C CNN
-F 1 "Conn_01x03" H 1018 1776 50  0000 C CNN
-F 2 "Connector2:JST_XH_B3B-XH-AM_1x03_P2.50mm_Vertical" H 1100 1550 50  0001 C CNN
-F 3 "~" H 1100 1550 50  0001 C CNN
-	1    1100 1550
-	-1   0    0    -1
-$EndComp
-$Comp
-L Connector_Generic:Conn_01x02 J?
-U 1 1 6035A4F8
-P 1100 2000
-AR Path="/6035A4F8" Ref="J?"  Part="1"
-AR Path="/60357CC4/6035A4F8" Ref="J4"  Part="1"
-F 0 "J4" H 1018 2217 50  0000 C CNN
-F 1 "Conn_01x02" H 1018 2126 50  0000 C CNN
-F 2 "Connector2:JST_XH_B2B-XH-AM_1x02_P2.50mm_Vertical" H 1100 2000 50  0001 C CNN
-F 3 "~" H 1100 2000 50  0001 C CNN
-	1    1100 2000
-	-1   0    0    -1
-$EndComp
 $Comp
 L Display2:SSD1306 U?
@@
 L power:VDC #PWR036
 U 1 1 6036C807
-P 1550 2000
-F 0 "#PWR036" H 1550 1900 50  0001 C CNN
-F 1 "VDC" H 1565 2173 50  0000 C CNN
-F 2 "" H 1550 2000 50  0001 C CNN
-F 3 "" H 1550 2000 50  0001 C CNN
-	1    1550 2000
+P 1100 1550
+F 0 "#PWR036" H 1100 1450 50  0001 C CNN
+F 1 "VDC" H 1115 1723 50  0000 C CNN
+F 2 "" H 1100 1550 50  0001 C CNN
+F 3 "" H 1100 1550 50  0001 C CNN
+	1    1100 1550
 	1    0    0    -1
 $EndComp
@@
 L power:GNDA #PWR037
 U 1 1 6036D122
-P 1550 2100
-F 0 "#PWR037" H 1550 1850 50  0001 C CNN
-F 1 "GNDA" H 1555 1927 50  0000 C CNN
-F 2 "" H 1550 2100 50  0001 C CNN
-F 3 "" H 1550 2100 50  0001 C CNN
-	1    1550 2100
-	1    0    0    -1
-$EndComp
-Wire Wire Line
-	1300 2000 1550 2000
-Wire Wire Line
-	1300 2100 1550 2100
+P 1100 1650
+F 0 "#PWR037" H 1100 1400 50  0001 C CNN
+F 1 "GNDA" H 1105 1477 50  0000 C CNN
+F 2 "" H 1100 1650 50  0001 C CNN
+F 3 "" H 1100 1650 50  0001 C CNN
+	1    1100 1650
+	1    0    0    -1
+$EndComp
 $Comp
 L power:GNDA #PWR041
@@
 Wire Wire Line
 	6400 1500 6250 1500
-Wire Wire Line
-	1300 1450 1500 1450
-Wire Wire Line
-	1300 1650 1500 1650
-Wire Wire Line
-	1300 1550 1750 1550
-Wire Wire Line
-	1750 1550 1750 2300
-Wire Wire Line
-	1750 2300 1900 2300
-Wire Wire Line
-	1500 1450 1500 1500
-Wire Wire Line
-	1500 1500 2150 1500
-Wire Wire Line
-	1500 1600 1500 1650
-Wire Wire Line
-	1500 1600 2150 1600
-Text Label 1350 1450 0    50   ~ 0
-SCL
-Text Label 1350 1650 0    50   ~ 0
-SDA
 $Comp
 L Mechanical:MountingHole_Pad H5
@@
 	1    0    0    -1
 $EndComp
-$Comp
-L power:GNDA #PWR048
-U 1 1 60391EC2
-P 6500 2800
-F 0 "#PWR048" H 6500 2550 50  0001 C CNN
-F 1 "GNDA" H 6505 2627 50  0000 C CNN
-F 2 "" H 6500 2800 50  0001 C CNN
-F 3 "" H 6500 2800 50  0001 C CNN
-	1    6500 2800
-	1    0    0    -1
-$EndComp
 Wire Wire Line
 	6050 2800 6350 2800
 Connection ~ 6350 2800
-Wire Wire Line
-	6350 2800 6500 2800
-Connection ~ 6500 2800
-Wire Wire Line
-	6500 2800 6650 2800
 Connection ~ 6650 2800
 Wire Wire Line
@@
 Wire Wire Line
 	3150 2200 3300 2200
+$Comp
+L Connector_Generic:Conn_02x03_Odd_Even J?
+U 1 1 6160983A
+P 1500 1550
+AR Path="/6160983A" Ref="J?"  Part="1"
+AR Path="/60357CC4/6160983A" Ref="J3"  Part="1"
+F 0 "J3" H 1550 1350 50  0000 C CNN
+F 1 "Din_02x03" H 1550 1750 50  0000 C CNN
+F 2 "Connector_IDC:IDC-Header_2x03_P2.54mm_Vertical" H 1500 1550 50  0001 C CNN
+F 3 "~" H 1500 1550 50  0001 C CNN
+	1    1500 1550
+	-1   0    0    -1
+$EndComp
+NoConn ~ 1200 1450
+Wire Wire Line
+	1100 1550 1200 1550
+Wire Wire Line
+	1100 1650 1200 1650
+Wire Wire Line
+	1700 1450 2000 1450
+Wire Wire Line
+	2000 1450 2000 1600
+Wire Wire Line
+	2000 1600 2150 1600
+Wire Wire Line
+	1700 1550 2100 1550
+Wire Wire Line
+	2100 1550 2100 1500
+Wire Wire Line
+	2100 1500 2150 1500
+Wire Wire Line
+	1700 1650 1700 2300
+Wire Wire Line
+	1700 2300 1900 2300
+Text Label 1750 1550 0    50   ~ 0
+SCL
+Text Label 1750 1450 0    50   ~ 0
+SDA
+Wire Wire Line
+	6500 2800 6650 2800
+Wire Wire Line
+	6350 2800 6500 2800
+Connection ~ 6500 2800
+$Comp
+L power:GNDA #PWR048
+U 1 1 60391EC2
+P 6500 2800
+F 0 "#PWR048" H 6500 2550 50  0001 C CNN
+F 1 "GNDA" H 6505 2627 50  0000 C CNN
+F 2 "" H 6500 2800 50  0001 C CNN
+F 3 "" H 6500 2800 50  0001 C CNN
+	1    6500 2800
+	1    0    0    -1
+$EndComp
 $EndSCHEMATC
